File: Hardware/prog1/prog1.kicad_pcb (KiCad board)
At the start: 2 copper layers, 17 x 22 mm, 6 parts, among them J1 Conn_01x02, SW1 SW_Push

Commit message: hardware done
Routing:
- net +3V3: track 0.00 -> 9.75 mm
- net GND: track 2.11 -> 7.06 mm
Changed lines of the file:
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@@
     (style (thickness 0.1) (arrow_length 1.27) (text_position_mode 0) (extension_height 0.58642) (extension_offset 0.5) keep_text_aligned)
   )
+  (segment (start 113.46 80) (end 111.3028 77.8428) (width 0.25) (layer "F.Cu") (net 1))
   (segment (start 112.3444 74.2696) (end 112.3444 74.9044) (width 0.25) (layer "F.Cu") (net 1))
+  (segment (start 111.3028 77.8428) (end 111.3028 75.946) (width 0.25) (layer "F.Cu") (net 1))
   (segment (start 112.3444 74.9044) (end 111.3028 75.946) (width 0.25) (layer "F.Cu") (net 1))
   (via (at 111.3028 75.946) (size 0.8) (drill 0.4) (layers "F.Cu" "B.Cu") (free) (net 1))
@@
   (segment (start 119.3292 68.8848) (end 119.3292 72.2376) (width 0.25) (layer "F.Cu") (net 3))
   (segment (start 118.618 72.9488) (end 118.7196 73.0504) (width 0.25) (layer "F.Cu") (net 3))
+  (segment (start 123 73.365) (end 122.635 73.365) (width 0.25) (layer "F.Cu") (net 4))
+  (segment (start 122.635 73.365) (end 116 80) (width 0.25) (layer "F.Cu") (net 4))
   (zone (net 4) (net_name "+3V3") (layer "F.Cu") (hatch edge 0.5)
     (connect_pads (clearance 0.5))
