File: Hardware/prog1/prog1.kicad_pcb (KiCad board)
At the start: 2 copper layers, 17 x 21 mm, 6 parts, among them J1 Conn_01x02, SW1 SW_Push

Commit message: firmware finished?
Parts:
- moved J1 0.67 mm to (104.4, 105.7)
Changed lines of the file:
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@@
       (outputformat 1)
       (mirror false)
-      (drillshape 1)
+      (drillshape 0)
       (scaleselection 1)
-      (outputdirectory "")
+      (outputdirectory "DFM/")
     )
   )
@@
   )
   (footprint "Connector_Molex:Molex_KK-254_AE-6410-02A_1x02_P2.54mm_Vertical" (layer "F.Cu")
-    (at 104.46 105)
+    (at 104.394 105.664)
     (descr "Molex KK-254 Interconnect System, old/engineering part number: AE-6410-02A example for new part number: 22-27-2021, 2 Pins (http://www.molex.com/pdm_docs/sd/022272021_sd.pdf), generated with kicad-footprint-generator")
     (tags "connector Molex KK-254 vertical")
@@
     (fp_line (start 3.81 2.88) (end 3.81 -2.92)
       (stroke (width 0.1) (type solid)) (layer "F.Fab"))
-    (pad "1" thru_hole roundrect (at 0 0) (size 1.74 2.19) (drill 1.19) (layers "*.Cu" "*.Mask") (roundrect_rratio 0.143678)
+    (pad "1" thru_hole roundrect (at 0 0) (size 1.74 2.19) (drill 1.19) (layers "*.Cu" "*.Mask") (roundrect_rratio 0.1436781609)
       (net 1 "GND") (pinfunction "Pin_1") (pintype "passive"))
     (pad "2" thru_hole oval (at 2.54 0) (size 1.74 2.19) (drill 1.19) (layers "*.Cu" "*.Mask")
