File: Hardware/prog1/prog1.kicad_sch (KiCad schematic)
At the start: 4 parts, among them J1 Conn_01x02, SW1 SW_Push

Commit message: finished prog1 layout
Parts:
- R1: footprint Resistor_SMD:R_0201_0603Metric_Pad0.64x0.40mm_HandSolder -> Resistor_SMD:R_0603_1608Metric_Pad0.98x0.95mm_HandSolder
Changed lines of the file:
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@@
 			)
 		)
-		(property "Footprint" "Resistor_SMD:R_0201_0603Metric_Pad0.64x0.40mm_HandSolder"
+		(property "Footprint" "Resistor_SMD:R_0603_1608Metric_Pad0.98x0.95mm_HandSolder"
 			(at 89.916 65.786 90)
 			(effects
