File: Hardware/prog1/prog1.kicad_sch (KiCad schematic)
At the start: 3 parts

Commit message: Firmware project finished again
Parts:
- removed BT1: Battery_Cell, symbol Device:Battery_Cell
- removed D1: LED, symbol Device:LED
- added D1: LED_RED, layout:LED_0603_Symbol_on_F.SilkS, symbol device:LED
- added J1: Conn_01x02, Connector_Molex:Molex_KK-254_AE-6410-02A_1x02_P2.54mm_Vertical, symbol Connector_Generic:Conn_01x02
- added SW1: SW_Push, Button_Switch_SMD:SW_DIP_SPSTx01_Slide_6.7x4.1mm_W8.61mm_P2.54mm_LowProfile, symbol Switch:SW_Push
- R1: value R_US -> 105; footprint (none) -> Resistor_SMD:R_0603_1608Metric_Pad0.98x0.95mm_HandSolder
Connections:
- net at R1.1: now also D1.2 (A)
- net at R1.2: now also SW1.2
- new net +3V3: J1.2 (Pin_2), SW1.1
- new net GND: D1.1 (K), J1.1 (Pin_1)
