File: Hardware/prog1/prog1_v0.0.kicad_sch (KiCad schematic)
At the start: 4 parts, among them J1 Conn_01x02, SW1 SW_Push

Commit message: edit LED footprint
Parts:
- R1: footprint Resistor_SMD:R_0603_1608Metric_Pad0.98x0.95mm_HandSolder -> Resistor_SMD:R_0603_1608Metric
Changed lines of the file:
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@@
 			)
 		)
-		(property "Footprint" "Resistor_SMD:R_0603_1608Metric_Pad0.98x0.95mm_HandSolder"
+		(property "Footprint" "Resistor_SMD:R_0603_1608Metric"
 			(at 72.39 43.18 0)
 			(effects
