File: Hardware/prog1/prog1.kicad_pcb.kicad_pcb (KiCad board)
At the start: 2 copper layers, 0 parts

Commit message: First hardware project
Parts:
- added D1: LED_GREEN, layout:LED_0603_Symbol_on_F.SilkS, F.Cu at (126.5, 83.0)
- added J1: Conn_01x02, Connector_Molex:Molex_KK-254_AE-6410-02A_1x02_P2.54mm_Vertical, F.Cu at (127.5, 87.8)
- added R1: 105 OHM, Resistor_SMD:R_0603_1608Metric_Pad0.98x0.95mm_HandSolder, F.Cu at (131.1, 83.0)
- added REF**: 3.2mm_M3, MountingHole:MountingHole_3.2mm_M3, F.Cu at (129.0, 77.2)
- added REF**: 3.2mm_M3, MountingHole:MountingHole_3.2mm_M3, F.Cu at (136.0, 91.2)
- added SW1: SW_Push, Button_Switch_SMD:SW_DIP_SPSTx01_Slide_6.7x4.1mm_W8.61mm_P2.54mm_LowProfile, F.Cu at (136.0, 81.4)
Routing:
- net Net-(R1-Pad1): track 0.00 -> 8.34 mm
- net Net-(D1-A): track 0.00 -> 2.83 mm
- net GND: track 0.00 -> 1.78 mm, vias 0 -> 1
- added copper zone on F.Cu, net +3V3
- added copper zone on B.Cu, net GND
Other:
- board outline added: 15.7 x 22 mm
