File: Hardware/Project1/Project1.kicad_sch (KiCad schematic)
At the start: 4 parts, among them J1 Conn_01x02, SW1 SW_Push

Commit message: finished the hardware project
Parts:
- D1: footprint (none) -> layout:LED_0603_Symbol_on_F.SilkS
- J1: footprint (none) -> Connector_Molex:Molex_KK-254_AE-6410-02A_1x02_P2.54mm_Vertical; MPN (none) -> 022272021
- R1: footprint (none) -> Resistor_SMD:R_0603_1608Metric_Pad0.98x0.95mm_HandSolder
- SW1: footprint (none) -> Button_Switch_SMD:SW_DIP_SPSTx01_Slide_6.7x4.1mm_W6.73mm_P2.54mm_LowProfile_JPin; MPN (none) -> 1825910-6
Other:
- moved on the sheet: J1
Changed lines of the file:
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@@
     (comment 1 "Designed by: Thomas Vigh")
   )
+  (junction (at 115.57 86.36) (diameter 0) (color 0 0 0 0)
+  )
   (junction (at 115.57 96.52) (diameter 0) (color 0 0 0 0)
   )
-  (junction (at 110.49 86.36) (diameter 0) (color 0 0 0 0)
+  (junction (at 115.57 87.63) (diameter 0) (color 0 0 0 0)
+  )
+  (junction (at 115.57 95.25) (diameter 0) (color 0 0 0 0)
   )
   (wire (pts (xy 143.51 86.36) (xy 143.51 87.63))
     (stroke (width 0) (type default))
   )
-  (wire (pts (xy 110.49 91.44) (xy 110.49 86.36))
-    (stroke (width 0) (type default))
-  )
-  (wire (pts (xy 115.57 93.98) (xy 115.57 96.52))
+  (wire (pts (xy 115.57 90.17) (xy 115.57 87.63))
+    (stroke (width 0) (type default))
+  )
+  (wire (pts (xy 110.49 92.71) (xy 115.57 92.71))
+    (stroke (width 0) (type default))
+  )
+  (wire (pts (xy 115.57 87.63) (xy 115.57 86.36))
+    (stroke (width 0) (type default))
+  )
+  (wire (pts (xy 115.57 92.71) (xy 115.57 95.25))
     (stroke (width 0) (type default))
   )
@@
     (stroke (width 0) (type default))
   )
+  (wire (pts (xy 110.49 90.17) (xy 115.57 90.17))
+    (stroke (width 0) (type default))
+  )
   (wire (pts (xy 143.51 95.25) (xy 143.51 96.52))
     (stroke (width 0) (type default))
   )
-  (wire (pts (xy 110.49 86.36) (xy 110.49 85.09))
-    (stroke (width 0) (type default))
-  )
-  (wire (pts (xy 107.95 91.44) (xy 110.49 91.44))
-    (stroke (width 0) (type default))
-  )
   (wire (pts (xy 139.7 86.36) (xy 143.51 86.36))
     (stroke (width 0) (type default))
   )
-  (wire (pts (xy 107.95 93.98) (xy 115.57 93.98))
-    (stroke (width 0) (type default))
-  )
   (wire (pts (xy 143.51 96.52) (xy 115.57 96.52))
     (stroke (width 0) (type default))
   )
-  (wire (pts (xy 110.49 86.36) (xy 118.11 86.36))
+  (wire (pts (xy 115.57 86.36) (xy 118.11 86.36))
+    (stroke (width 0) (type default))
+  )
+  (wire (pts (xy 115.57 85.09) (xy 115.57 86.36))
+    (stroke (width 0) (type default))
+  )
+  (wire (pts (xy 115.57 95.25) (xy 115.57 96.52))
     (stroke (width 0) (type default))
   )
@@
     (pin "1")
     (instances
-      (project "Project1.kicad_pro"
+      (project "Project1"
         (path "/f7e68b08-6f2b-4c78-ad38-5fdd6a11b185"
           (reference "#PWR02") (unit 1)
@@
       (effects (font (size 1.27 1.27)) (justify right))
     )
-    (property "Footprint" "" (at 143.51 91.44 0)
+    (property "Footprint" "layout:LED_0603_Symbol_on_F.SilkS" (at 143.51 91.44 0)
       (effects (font (size 1.27 1.27)) hide)
     )
@@
       (effects (font (size 1.27 1.27)) hide)
     )
-    (pin "1")
-    (pin "2")
-    (instances
-      (project "Project1.kicad_pro"
+    (property "MPN" "" (at 143.51 91.44 0)
+      (effects (font (size 1.27 1.27)) hide)
+    )
+    (property "Notes" "" (at 143.51 91.44 0)
+      (effects (font (size 1.27 1.27)) hide)
+    )
+    (pin "1")
+    (pin "2")
+    (instances
+      (project "Project1"
         (path "/f7e68b08-6f2b-4c78-ad38-5fdd6a11b185"
           (reference "D1") (unit 1)
@@
     )
   )
+  (symbol (lib_id "power:PWR_FLAG") (at 115.57 95.25 90) (unit 1)
+    (in_bom yes) (on_board yes) (dnp no)
+    (property "Reference" "#FLG02" (at 113.665 95.25 0)
+      (effects (font (size 1.27 1.27)) hide)
+    )
+    (property "Value" "PWR_FLAG" (at 111.76 102.87 0)
+      (effects (font (size 1.27 1.27)) (justify left))
+    )
+    (property "Footprint" "" (at 115.57 95.25 0)
+      (effects (font (size 1.27 1.27)) hide)
+    )
+    (property "Datasheet" "~" (at 115.57 95.25 0)
+      (effects (font (size 1.27 1.27)) hide)
+    )
+    (pin "1")
+    (instances
+      (project "Project1"
+        (path "/f7e68b08-6f2b-4c78-ad38-5fdd6a11b185"
+          (reference "#FLG02") (unit 1)
+        )
+      )
+    )
+  )
   (symbol (lib_id "Device:R") (at 135.89 86.36 90) (unit 1)
     (in_bom yes) (on_board yes) (dnp no) (fields_autoplaced)
@@
       (effects (font (size 1.27 1.27)))
     )
-    (property "Footprint" "" (at 135.89 88.138 90)
+    (property "Footprint" "Resistor_SMD:R_0603_1608Metric_Pad0.98x0.95mm_HandSolder" (at 135.89 88.138 90)
       (effects (font (size 1.27 1.27)) hide)
     )
@@
       (effects (font (size 1.27 1.27)) hide)
     )
-    (pin "1")
-    (pin "2")
-    (instances
-      (project "Project1.kicad_pro"
+    (property "MPN" "" (at 135.89 86.36 0)
+      (effects (font (size 1.27 1.27)) hide)
+    )
+    (property "Notes" "" (at 135.89 86.36 0)
+      (effects (font (size 1.27 1.27)) hide)
+    )
+    (pin "1")
+    (pin "2")
+    (instances
+      (project "Project1"
         (path "/f7e68b08-6f2b-4c78-ad38-5fdd6a11b185"
           (reference "R1") (unit 1)
@@
     )
   )
+  (symbol (lib_id "power:PWR_FLAG") (at 115.57 87.63 90) (unit 1)
+    (in_bom yes) (on_board yes) (dnp no)
+    (property "Reference" "#FLG01" (at 113.665 87.63 0)
+      (effects (font (size 1.27 1.27)) hide)
+    )
+    (property "Value" "PWR_FLAG" (at 111.76 90.17 0)
+      (effects (font (size 1.27 1.27)) (justify left))
+    )
+    (property "Footprint" "" (at 115.57 87.63 0)
+      (effects (font (size 1.27 1.27)) hide)
+    )
+    (property "Datasheet" "~" (at 115.57 87.63 0)
+      (effects (font (size 1.27 1.27)) hide)
+    )
+    (pin "1")
+    (instances
+      (project "Project1"
+        (path "/f7e68b08-6f2b-4c78-ad38-5fdd6a11b185"
+          (reference "#FLG01") (unit 1)
+        )
+      )
+    )
+  )
   (symbol (lib_id "Switch:SW_Push") (at 123.19 86.36 0) (unit 1)
     (in_bom yes) (on_board yes) (dnp no) (fields_autoplaced)
@@
       (effects (font (size 1.27 1.27)))
     )
-    (property "Footprint" "" (at 123.19 81.28 0)
-      (effects (font (size 1.27 1.27)) hide)
-    )
-    (property "Datasheet" "~" (at 123.19 81.28 0)
-      (effects (font (size 1.27 1.27)) hide)
-    )
-    (pin "1")
-    (pin "2")
-    (instances
-      (project "Project1.kicad_pro"
+    (property "Footprint" "Button_Switch_SMD:SW_DIP_SPSTx01_Slide_6.7x4.1mm_W6.73mm_P2.54mm_LowProfile_JPin" (at 123.19 81.28 0)
+      (effects (font (size 1.27 1.27)) hide)
+    )
+    (property "Datasheet" "https://www.digikey.com/en/products/detail/te-connectivity-alcoswitch-switches/1825910-6/1632536?utm_adgroup=Supplier_TE&utm_source=google&utm_medium=cpc&utm_campaign=EN_Product_SKU_MBR&utm_term=%2B1825910-6&utm_content=Supplier_TE&gclid=Cj0KCQjwp4j6BRCRARIsAGq4yMGhBEsv1v5KcRzgW34aOMlPkoRB4A-7BCN08FfGaiq_Dk_nlKJ0QU8aAhZPEALw_wcB" (at 123.19 81.28 0)
+      (effects (font (size 1.27 1.27)) hide)
+    )
+    (property "MPN" "1825910-6" (at 123.19 86.36 0)
+      (effects (font (size 1.27 1.27)) hide)
+    )
+    (property "Notes" "" (at 123.19 86.36 0)
+      (effects (font (size 1.27 1.27)) hide)
+    )
+    (pin "1")
+    (pin "2")
+    (instances
+      (project "Project1"
         (path "/f7e68b08-6f2b-4c78-ad38-5fdd6a11b185"
           (reference "SW1") (unit 1)
@@
     )
   )
-  (symbol (lib_id "Connector_Generic:Conn_01x02") (at 102.87 93.98 180) (unit 1)
-    (in_bom yes) (on_board yes) (dnp no) (fields_autoplaced)
-    (property "Reference" "J1" (at 102.87 85.09 0)
-      (effects (font (size 1.27 1.27)))
-    )
-    (property "Value" "Conn_01x02" (at 102.87 87.63 0)
-      (effects (font (size 1.27 1.27)))
-    )
-    (property "Footprint" "" (at 102.87 93.98 0)
-      (effects (font (size 1.27 1.27)) hide)
-    )
-    (property "Datasheet" "~" (at 102.87 93.98 0)
-      (effects (font (size 1.27 1.27)) hide)
-    )
-    (pin "1")
-    (pin "2")
-    (instances
-      (project "Project1.kicad_pro"
+  (symbol (lib_id "Connector_Generic:Conn_01x02") (at 105.41 92.71 180) (unit 1)
+    (in_bom yes) (on_board yes) (dnp no)
+    (property "Reference" "J1" (at 99.06 91.44 90)
+      (effects (font (size 1.27 1.27)))
+    )
+    (property "Value" "Conn_01x02" (at 101.6 91.44 90)
+      (effects (font (size 1.27 1.27)))
+    )
+    (property "Footprint" "Connector_Molex:Molex_KK-254_AE-6410-02A_1x02_P2.54mm_Vertical" (at 105.41 92.71 0)
+      (effects (font (size 1.27 1.27)) hide)
+    )
+    (property "Datasheet" "https://tools.molex.com/pdm_docs/sd/022272021_sd.pdf" (at 105.41 92.71 0)
+      (effects (font (size 1.27 1.27)) hide)
+    )
+    (property "MPN" "022272021" (at 105.41 92.71 0)
+      (effects (font (size 1.27 1.27)) hide)
+    )
+    (property "Notes" "" (at 105.41 92.71 0)
+      (effects (font (size 1.27 1.27)) hide)
+    )
+    (pin "1")
+    (pin "2")
+    (instances
+      (project "Project1"
         (path "/f7e68b08-6f2b-4c78-ad38-5fdd6a11b185"
           (reference "J1") (unit 1)
@@
     )
   )
-  (symbol (lib_id "power:+3V3") (at 110.49 85.09 0) (unit 1)
-    (in_bom yes) (on_board yes) (dnp no) (fields_autoplaced)
-    (property "Reference" "#PWR01" (at 110.49 88.9 0)
-      (effects (font (size 1.27 1.27)) hide)
-    )
-    (property "Value" "+3V3" (at 110.49 80.01 0)
-      (effects (font (size 1.27 1.27)))
-    )
-    (property "Footprint" "" (at 110.49 85.09 0)
-      (effects (font (size 1.27 1.27)) hide)
-    )
-    (property "Datasheet" "" (at 110.49 85.09 0)
-      (effects (font (size 1.27 1.27)) hide)
-    )
-    (pin "1")
-    (instances
-      (project "Project1.kicad_pro"
+  (symbol (lib_id "power:+3V3") (at 115.57 85.09 0) (unit 1)
+    (in_bom yes) (on_board yes) (dnp no) (fields_autoplaced)
+    (property "Reference" "#PWR01" (at 115.57 88.9 0)
+      (effects (font (size 1.27 1.27)) hide)
+    )
+    (property "Value" "+3V3" (at 115.57 80.01 0)
+      (effects (font (size 1.27 1.27)))
+    )
+    (property "Footprint" "" (at 115.57 85.09 0)
+      (effects (font (size 1.27 1.27)) hide)
+    )
+    (property "Datasheet" "" (at 115.57 85.09 0)
+      (effects (font (size 1.27 1.27)) hide)
+    )
+    (pin "1")
+    (instances
+      (project "Project1"
         (path "/f7e68b08-6f2b-4c78-ad38-5fdd6a11b185"
           (reference "#PWR01") (unit 1)
