File: Hardware/p1 - Copy/p1.kicad_pcb (KiCad board)
At the start: 2 copper layers, 0 parts

Commit message: project finished with minor changes, pwr input is now a throughole component
Parts:
- added D1: LED, layout:LED_0603_Symbol_on_F.SilkS, F.Cu at (100.8, 58.4)
- added J1: Conn_01x02, layout:Molex_KK-254_1x02_P2.54mm_Horizontal, F.Cu at (102.9, 64.6)
- added R1: 105, Resistor_SMD:R_0603_1608Metric_Pad0.98x0.95mm_HandSolder, F.Cu at (105.8, 58.4)
- added REF**: MountingHole_3.2mm_M3, MountingHole:MountingHole_3.2mm_M3, F.Cu at (112.0, 72.0)
- added REF**: MountingHole_3.2mm_M3, MountingHole:MountingHole_3.2mm_M3, F.Cu at (104.1, 50.8)
- added SW1: SW_Push, Button_Switch_SMD:SW_DIP_SPSTx01_Slide_6.7x4.1mm_W6.73mm_P2.54mm_LowProfile_JPin, F.Cu at (111.8, 61.0)
Routing:
- net Net-(R1-Pad1): track 0.00 -> 10.1 mm
- net Net-(D1-A): track 0.00 -> 8.44 mm
- net +3V3: track 0.00 -> 6.49 mm
- net GND: track 0.00 -> 3.58 mm, vias 0 -> 1
- added copper zone on F.Cu, net +3V3
- added copper zone on B.Cu, net GND
Other:
- board outline added: 20 x 41 mm
