File: Hardware/Horn_Jake/Horn_Jake.kicad_sch (KiCad schematic)
At the start: 0 parts

Commit message: Horn Schematic and Layout
Parts:
- added C1, C2, C3, C4: .1 uF, Capacitor_SMD:CP_Elec_4x3, symbol Device:C
- added C5, C6: 1 uF, Capacitor_SMD:CP_Elec_4x5.4, symbol Device:C
- added C7, C8: 10 uF, Capacitor_SMD:CP_Elec_5x4.4, symbol Device:C
- added C9: 100 uF, Capacitor_SMD:CP_Elec_5x5.9, symbol device:C_Polarized_US
- added D1: Rectifier Diode, Diode_SMD:D_3220_8050Metric_Pad2.65x5.15mm_HandSolder, symbol pspice:DIODE
- added D2: Debug LED1, layout:LED_0603_Symbol_on_F.SilkS, symbol device:LED
- added D3: Debug LED2, layout:LED_0603_Symbol_on_F.SilkS, symbol device:LED
- added D4: Debug LED3, layout:LED_0603_Symbol_on_F.SilkS, symbol device:LED
- added F1: 2A, Fuse:Fuse_0603_1608Metric_Pad1.05x0.95mm_HandSolder, symbol device:Fuse
- added J1: Horn 1, Connector_Molex:Molex_KK-254_AE-6410-02A_1x02_P2.54mm_Vertical, symbol Connector_Generic:Conn_01x02
- added J2: Horn 2, Connector_Molex:Molex_KK-254_AE-6410-02A_1x02_P2.54mm_Vertical, symbol Connector_Generic:Conn_01x02
- added J3: Horn Control, Connector_Molex:Molex_KK-254_AE-6410-02A_1x02_P2.54mm_Vertical, symbol Connector_Generic:Conn_01x02
- added J4: Power, Connector_Molex:Molex_KK-254_AE-6410-03A_1x03_P2.54mm_Vertical, symbol Connector_Generic:Conn_01x03
- added Q1: N-type transistor, Package_TO_SOT_THT:TO-92L_HandSolder, symbol Device:Q_NUJT_BEB
- added R1: 1000 ohm, Resistor_SMD:R_0603_1608Metric_Pad0.98x0.95mm_HandSolder, symbol Device:R_US
- added SW1: Debug Switch, Button_Switch_SMD:SW_DIP_SPSTx01_Slide_6.7x4.1mm_W8.61mm_P2.54mm_LowProfile, symbol Switch:SW_Push
Connections:
- new net: D1.2 (A), J2.1 (Pin_1)
- new net: J1.1 (Pin_1), J2.2 (Pin_2)
- new net: C2.2, C3.2, C4.2, C5.2, C6.2, C7.2, C8.2, C9.2, D1.1 (K)
- new net: C1.2, R1.2
- new net: F1.1, Q1.3 (B1), SW1.1
- new net: D3.1 (K), F1.2
- new net: D2.2 (A), J4.2 (Pin_2)
- new net: D4.2 (A), J3.1 (Pin_1)
- new net: C1.1, J3.2 (Pin_2)
- new net +24V: C2.1, C3.1, C4.1, C5.1, C6.1, C7.1, C8.1, C9.1, D2.1 (K)
- new net GND: J4.1 (Pin_1), J4.3 (Pin_3), Q1.1 (B2), R1.1, SW1.2
- new net HORN_CTL: D4.1 (K), Q1.2 (E)
- new net HORN_IN: D3.2 (A), J1.2 (Pin_2)

Commit message: Hardware Advanced Project Completion
Connections:
- net +24V: now also D2.2 (A), J4.2 (Pin_2); no longer C2.1, C3.1, C4.1, C5.1, C6.1, C7.1, C8.1, C9.1, D2.1 (K)
- new net: C2.1, C3.1, C4.1, C5.1, C6.1, C7.1, C8.1, C9.1, D2.1 (K)
Other:
- moved on the sheet: D2, J4
Changed lines of the file:
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@@
   (junction (at 71.374 81.28) (diameter 0) (color 0 0 0 0)
   )
-  (junction (at 117.856 63.5) (diameter 0) (color 0 0 0 0)
-  )
   (junction (at 131.445 76.835) (diameter 0) (color 0 0 0 0)
   )
@@
   (junction (at 123.825 69.85) (diameter 0) (color 0 0 0 0)
   )
+  (junction (at 117.856 76.073) (diameter 0) (color 0 0 0 0)
+  )
   (junction (at 113.03 79.502) (diameter 0) (color 0 0 0 0)
   )
@@
     (stroke (width 0) (type default))
   )
+  (wire (pts (xy 115.57 76.073) (xy 117.856 76.073))
+    (stroke (width 0) (type default))
+  )
   (wire (pts (xy 131.445 48.895) (xy 131.445 55.88))
     (stroke (width 0) (type default))
@@
     (stroke (width 0) (type default))
   )
+  (wire (pts (xy 99.822 86.36) (xy 102.87 86.36))
+    (stroke (width 0) (type default))
+  )
   (wire (pts (xy 131.445 69.85) (xy 131.445 76.835))
     (stroke (width 0) (type default))
@@
     (stroke (width 0) (type default))
   )
-  (wire (pts (xy 117.856 63.5) (xy 117.856 76.2))
+  (wire (pts (xy 117.856 63.5) (xy 117.856 65.659))
     (stroke (width 0) (type default))
   )
@@
     (stroke (width 0) (type default))
   )
+  (wire (pts (xy 115.57 63.5) (xy 115.57 76.073))
+    (stroke (width 0) (type default))
+  )
   (wire (pts (xy 113.03 79.375) (xy 113.03 79.502))
     (stroke (width 0) (type default))
@@
     (stroke (width 0) (type default))
   )
-  (wire (pts (xy 99.822 86.36) (xy 102.362 86.36))
-    (stroke (width 0) (type default))
-  )
   (wire (pts (xy 131.445 104.14) (xy 120.65 104.14))
     (stroke (width 0) (type default))
@@
     (stroke (width 0) (type default))
   )
-  (wire (pts (xy 117.856 83.82) (xy 117.856 91.694))
+  (wire (pts (xy 117.856 76.073) (xy 117.856 91.694))
+    (stroke (width 0) (type default))
+  )
+  (wire (pts (xy 102.362 83.82) (xy 102.87 83.82))
     (stroke (width 0) (type default))
   )
@@
     (stroke (width 0) (type default))
   )
-  (wire (pts (xy 115.57 63.5) (xy 117.856 63.5))
-    (stroke (width 0) (type default))
-  )
   (wire (pts (xy 82.55 81.28) (xy 90.17 81.28))
     (stroke (width 0) (type default))
@@
   )
   (wire (pts (xy 123.825 62.865) (xy 123.825 63.5))
+    (stroke (width 0) (type default))
+  )
+  (wire (pts (xy 117.856 73.279) (xy 117.856 76.073))
+    (stroke (width 0) (type default))
+  )
+  (wire (pts (xy 102.362 88.9) (xy 102.87 88.9))
     (stroke (width 0) (type default))
   )
@@
       (effects (font (size 1.27 1.27)) hide)
     )
-    (property "Datasheet" "~" (at 92.71 93.98 0)
+    (property "Datasheet" "https://www.mouser.com/datasheet/2/115/diodes%20inc._ds14002-1163889.pdf" (at 92.71 93.98 0)
       (effects (font (size 1.27 1.27)) hide)
     )
@@
     )
   )
-  (symbol (lib_id "device:LED") (at 117.856 80.01 270) (unit 1)
+  (symbol (lib_id "device:LED") (at 117.856 69.469 270) (unit 1)
     (in_bom yes) (on_board yes) (dnp no) (fields_autoplaced)
-    (property "Reference" "D2" (at 120.65 77.1525 90)
-      (effects (font (size 1.27 1.27)) (justify left))
-    )
-    (property "Value" "Debug LED1" (at 120.65 79.6925 90)
-      (effects (font (size 1.27 1.27)) (justify left))
-    )
-    (property "Footprint" "layout:LED_0603_Symbol_on_F.SilkS" (at 117.856 80.01 0)
-      (effects (font (size 1.27 1.27)) hide)
-    )
-    (property "Datasheet" "~" (at 117.856 80.01 0)
+    (property "Reference" "D2" (at 120.523 66.6115 90)
+      (effects (font (size 1.27 1.27)) (justify left))
+    )
+    (property "Value" "Debug LED1" (at 120.523 69.1515 90)
+      (effects (font (size 1.27 1.27)) (justify left))
+    )
+    (property "Footprint" "layout:LED_0603_Symbol_on_F.SilkS" (at 117.856 69.469 0)
+      (effects (font (size 1.27 1.27)) hide)
+    )
+    (property "Datasheet" "~" (at 117.856 69.469 0)
       (effects (font (size 1.27 1.27)) hide)
     )
@@
       (effects (font (size 1.27 1.27)) hide)
     )
-    (property "Datasheet" "~" (at 97.536 67.818 0)
+    (property "Datasheet" "https://www.vishay.com/docs/45171/kseries.pdf" (at 97.536 67.818 0)
       (effects (font (size 1.27 1.27)) hide)
     )
@@
       (effects (font (size 1.27 1.27)) hide)
     )
-    (property "Datasheet" "~" (at 127.635 62.865 0)
+    (property "Datasheet" "https://www.vishay.com/docs/45171/kseries.pdf" (at 127.635 62.865 0)
       (effects (font (size 1.27 1.27)) hide)
     )
@@
       (effects (font (size 1.27 1.27)) hide)
     )
-    (property "Datasheet" "~" (at 127.635 55.88 0)
+    (property "Datasheet" "https://www.vishay.com/docs/45171/kseries.pdf" (at 127.635 55.88 0)
       (effects (font (size 1.27 1.27)) hide)
     )
@@
       (effects (font (size 1.27 1.27)) hide)
     )
-    (property "Datasheet" "~" (at 76.454 78.74 0)
+    (property "Datasheet" "https://www.vishay.com/docs/91420/sihfr010.pdf" (at 76.454 78.74 0)
       (effects (font (size 1.27 1.27)) hide)
     )
@@
       (effects (font (size 1.27 1.27)) hide)
     )
-    (property "Datasheet" "~" (at 127.635 98.425 0)
+    (property "Datasheet" "https://www.vishay.com/docs/28316/116rll.pdf" (at 127.635 98.425 0)
       (effects (font (size 1.27 1.27)) hide)
     )
@@
       (effects (font (size 1.27 1.27)) hide)
     )
-    (property "Datasheet" "~" (at 127.635 48.895 0)
+    (property "Datasheet" "https://www.vishay.com/docs/45171/kseries.pdf" (at 127.635 48.895 0)
       (effects (font (size 1.27 1.27)) hide)
     )
@@
     )
   )
-  (symbol (lib_id "Connector_Generic:Conn_01x03") (at 107.442 86.36 0) (unit 1)
+  (symbol (lib_id "Connector_Generic:Conn_01x03") (at 107.95 86.36 0) (unit 1)
     (in_bom yes) (on_board yes) (dnp no) (fields_autoplaced)
-    (property "Reference" "J4" (at 110.617 85.09 0)
-      (effects (font (size 1.27 1.27)) (justify left))
-    )
-    (property "Value" "Power" (at 110.617 87.63 0)
-      (effects (font (size 1.27 1.27)) (justify left))
-    )
-    (property "Footprint" "Connector_Molex:Molex_KK-254_AE-6410-03A_1x03_P2.54mm_Vertical" (at 107.442 86.36 0)
-      (effects (font (size 1.27 1.27)) hide)
-    )
-    (property "Datasheet" "~" (at 107.442 86.36 0)
-      (effects (font (size 1.27 1.27)) hide)
-    )
+    (property "Reference" "J4" (at 111.125 85.09 0)
+      (effects (font (size 1.27 1.27)) (justify left))
+    )
+    (property "Value" "Power" (at 111.125 87.63 0)
+      (effects (font (size 1.27 1.27)) (justify left))
+    )
+    (property "Footprint" "Connector_Molex:Molex_KK-254_AE-6410-03A_1x03_P2.54mm_Vertical" (at 107.95 86.36 0)
+      (effects (font (size 1.27 1.27)) hide)
+    )
+    (property "Datasheet" "~" (at 107.95 86.36 0)
+      (effects (font (size 1.27 1.27)) hide)
+    )
