File: Hardware/hornsBoard/hornsBoard.kicad_pcb (KiCad board)
At the start: 2 copper layers, 0 parts

Commit message: Hardware Project 2 Complete
Parts:
- added C1: C, Capacitor_SMD:C_0603_1608Metric_Pad1.08x0.95mm_HandSolder, F.Cu at (143.8, 113.0)
- added F1: 2A, Fuse:Fuse_0603_1608Metric_Pad1.05x0.95mm_HandSolder, F.Cu at (143.5, 107.2)
- added J1: Conn_01x03, Connector_Molex:Molex_KK-254_AE-6410-03A_1x03_P2.54mm_Vertical, F.Cu at (150.8, 119.0)
- added J2: Conn_01x02, Connector_Molex:Molex_KK-254_AE-6410-02A_1x02_P2.54mm_Vertical, F.Cu at (157.5, 109.5)
- added J3: Conn_01x02, Connector_Molex:Molex_KK-254_AE-6410-02A_1x02_P2.54mm_Vertical, F.Cu at (156.0, 102.0)
- added J4: Conn_01x02, Connector_Molex:Molex_KK-254_AE-6410-02A_1x02_P2.54mm_Vertical, F.Cu at (148.5, 102.0)
- added Q2: IRF6785, Package_DirectFET:DirectFET_MZ, F.Cu at (149.8, 111.0)
- added R1: R_US, Resistor_SMD:R_0603_1608Metric_Pad0.98x0.95mm_HandSolder, F.Cu at (143.8, 110.2)
- added REF**: MountingHole_3.2mm_M3, MountingHole:MountingHole_3.2mm_M3, F.Cu at (142.0, 101.0)
- added REF**: MountingHole_3.2mm_M3, MountingHole:MountingHole_3.2mm_M3, F.Cu at (158.0, 120.0)
Routing:
- net /Horn_Signal: track 0.00 -> 25.9 mm
- net GND: track 0.00 -> 7.58 mm, vias 0 -> 3
- net Net-(Q2-G): track 0.00 -> 7.04 mm
- net Net-(J4-Pin_1): track 0.00 -> 6.77 mm
- net Net-(J3-Pin_1): track 0.00 -> 4.96 mm
- added copper zone on F.Cu, net /24V
- added copper zone on B.Cu, net GND
Other:
- board outline added: 24 x 27 mm
- board text added: "Horn Control Board"
- board text added: "HornIn"
- board text added: "HornOut"
- board text added: "Power"
