File: Hardware/hornsBoard/hornsBoard.kicad_sch (KiCad schematic)
At the start: 0 parts

Commit message: Hardware Project 2 Complete
Parts:
- added C1: C, Capacitor_SMD:C_0603_1608Metric_Pad1.08x0.95mm_HandSolder, symbol Device:C
- added F1: 2A, Fuse:Fuse_0603_1608Metric_Pad1.05x0.95mm_HandSolder, symbol device:Fuse
- added J1: Conn_01x03, Connector_Molex:Molex_KK-254_AE-6410-03A_1x03_P2.54mm_Vertical, symbol Connector_Generic:Conn_01x03
- added J2, J3, J4: Conn_01x02, Connector_Molex:Molex_KK-254_AE-6410-02A_1x02_P2.54mm_Vertical, symbol Connector_Generic:Conn_01x02
- added Q2: IRF6785, Package_DirectFET:DirectFET_MZ, symbol Transistor_FET:IRF6785
- added R1: R_US, Resistor_SMD:R_0603_1608Metric_Pad0.98x0.95mm_HandSolder, symbol Device:R_US
Connections:
- new net: F1.1, J4.1 (Pin_1)
- new net: F1.2, Q2.2 (G)
- new net: J3.1 (Pin_1), J4.2 (Pin_2)
- new net 24V: J1.2 (Pin_2), J3.2 (Pin_2)
- new net GND: C1.2, J1.1 (Pin_1), J1.3 (Pin_3), J2.1 (Pin_1), Q2.3 (S), R1.2
- new net Horn_Signal: C1.1, J2.2 (Pin_2), Q2.1 (D), R1.1
Other:
- note added: "Horn Control"
- note added: "Horn Out"
- note added: "Power"
- title: Template -> Horns Board
