File: Hardware/aryano2_Horns_v1.0./Horns_v1.0.kicad_sch (KiCad schematic)
At the start: 0 parts

Commit message: horns_v.1.0 schematic done
Parts:
- added C2: 21 u, symbol Device:C
- added C3: 210 u, symbol Device:C
- added C4: 3.1 u, symbol Device:C
- added C5: C, symbol Device:C
- added C6: 1100 u, symbol device:C_Polarized_US
- added D1: ESD9B5.0ST5G, Diode_SMD:D_SOD-923, symbol Diode:ESD9B5.0ST5G
- added F1: 2A, symbol device:Fuse
- added J1, J3, J4: Conn_01x02_Female, symbol Connector:Conn_01x02_Female
- added J2: Conn_01x03_Female, symbol Connector:Conn_01x03_Female
- added Q1: IRLIZ44N, Package_TO_SOT_THT:TO-220F-3_Vertical, symbol Transistor_FET:IRLIZ44N
- added R2: R, symbol device:R
Connections:
- new net: C5.2, R2.1
- new net: J1.2 (Pin_2), J3.1 (Pin_1)
- new net: F1.1, Q1.2 (D)
- new net +24V: C2.1, C3.1, C4.1, C6.1, D1.2 (A2), J2.2 (Pin_2), J3.2 (Pin_2)
- new net GND: C2.2, C3.2, C4.2, C6.2, J2.1 (Pin_1), J2.3 (Pin_3), J4.1 (Pin_1), Q1.3 (S), R2.2
- new net HORN_CTRL: C5.1, J4.2 (Pin_2), Q1.1 (G)
- new net HORN_IN: D1.1 (A1), F1.2, J1.1 (Pin_1)

Commit message: added footprints to schematic
Parts:
- C2, C3, C4, C5, C6: footprint (none) -> Capacitor_SMD:C_1206_3216Metric
- F1: footprint (none) -> Fuse:Fuse_1206_3216Metric
- J1, J3, J4: footprint (none) -> Connector_PinSocket_2.54mm:PinSocket_1x02_P2.54mm_Vertical
- J2: footprint (none) -> Connector_PinSocket_2.54mm:PinSocket_1x03_P2.54mm_Vertical
- R2: footprint (none) -> Resistor_SMD:R_1206_3216Metric
Changed lines of the file:
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@@
       (effects (font (size 1.27 1.27)))
     )
-    (property "Footprint" "" (at 69.85 94.488 90)
+    (property "Footprint" "Resistor_SMD:R_1206_3216Metric" (at 69.85 94.488 90)
       (effects (font (size 1.27 1.27)) hide)
     )
@@
       (effects (font (size 1.27 1.27)) (justify right))
     )
-    (property "Footprint" "" (at 123.19 60.96 0)
+    (property "Footprint" "Connector_PinSocket_2.54mm:PinSocket_1x02_P2.54mm_Vertical" (at 123.19 60.96 0)
       (effects (font (size 1.27 1.27)) hide)
     )
@@
       (effects (font (size 1.27 1.27)))
     )
-    (property "Footprint" "" (at 105.41 69.088 90)
+    (property "Footprint" "Fuse:Fuse_1206_3216Metric" (at 105.41 69.088 90)
       (effects (font (size 1.27 1.27)) hide)
     )
@@
       (effects (font (size 1.27 1.27)) (justify left))
     )
-    (property "Footprint" "" (at 134.62 103.1748 0)
+    (property "Footprint" "Capacitor_SMD:C_1206_3216Metric" (at 134.62 103.1748 0)
       (effects (font (size 1.27 1.27)) hide)
     )
@@
       (effects (font (size 1.27 1.27)) (justify left))
     )
-    (property "Footprint" "" (at 66.04 58.42 0)
+    (property "Footprint" "Connector_PinSocket_2.54mm:PinSocket_1x03_P2.54mm_Vertical" (at 66.04 58.42 0)
       (effects (font (size 1.27 1.27)) hide)
     )
@@
       (effects (font (size 1.27 1.27)))
     )
-    (property "Footprint" "" (at 60.96 91.7448 0)
+    (property "Footprint" "Capacitor_SMD:C_1206_3216Metric" (at 60.96 91.7448 0)
       (effects (font (size 1.27 1.27)) hide)
     )
@@
       (effects (font (size 1.27 1.27)) (justify right))
     )
-    (property "Footprint" "" (at 123.19 50.8 0)
+    (property "Footprint" "Connector_PinSocket_2.54mm:PinSocket_1x02_P2.54mm_Vertical" (at 123.19 50.8 0)
       (effects (font (size 1.27 1.27)) hide)
     )
@@
       (effects (font (size 1.27 1.27)) (justify left))
     )
-    (property "Footprint" "" (at 134.62 98.0948 0)
+    (property "Footprint" "Capacitor_SMD:C_1206_3216Metric" (at 134.62 98.0948 0)
       (effects (font (size 1.27 1.27)) hide)
     )
@@
       (effects (font (size 1.27 1.27)))
     )
-    (property "Footprint" "" (at 129.54 110.49 0)
+    (property "Footprint" "Capacitor_SMD:C_1206_3216Metric" (at 129.54 110.49 0)
       (effects (font (size 1.27 1.27)) hide)
     )
@@
       (effects (font (size 1.27 1.27)) (justify left))
     )
-    (property "Footprint" "" (at 134.62 93.0148 0)
+    (property "Footprint" "Capacitor_SMD:C_1206_3216Metric" (at 134.62 93.0148 0)
       (effects (font (size 1.27 1.27)) hide)
     )
@@
       (effects (font (size 1.27 1.27)) (justify right))
     )
-    (property "Footprint" "" (at 86.36 45.72 0)
-      (effects (font (size 1.27 1.27)) hide)
-    )
+    (property "Footprint" "Connector_PinSocket_2.54mm:PinSocket_1x02_P2.54mm_Vertical" (at 86.36 45.72 0)
+      (effects (font (size 1.27 1.27)) hide)
+    )

Commit message: final , finished hardware project 2
Parts:
- removed J1, J3, J4: Conn_01x02_Female, Connector_PinSocket_2.54mm:PinSocket_1x02_P2.54mm_Vertical, symbol Connector:Conn_01x02_Female
- removed J2: Conn_01x03_Female, Connector_PinSocket_2.54mm:PinSocket_1x03_P2.54mm_Vertical, symbol Connector:Conn_01x03_Female
- added J1, J2, J5: Conn_01x02, Connector_Molex:Molex_Micro-Fit_3.0_43650-0200_1x02_P3.00mm_Horizontal, symbol Connector_Generic:Conn_01x02
- added J3: Conn_01x03, Connector_Molex:Molex_Micro-Fit_3.0_43650-0300_1x03_P3.00mm_Horizontal, symbol Connector_Generic:Conn_01x03
Connections:
- net +24V: now also J1.2 (Pin_2), J3.2 (Pin_2)
- net GND: now also J2.1 (Pin_1), J3.1 (Pin_1), J3.3 (Pin_3)
- net HORN_CTRL: now also J2.2 (Pin_2)
- net HORN_IN: now also J5.1 (Pin_1)
- new net: J1.1 (Pin_1), J5.2 (Pin_2)
