File: Hardware/Dev/Template_v0.0/LED/LED.kicad_pcb (KiCad board)
At the start: 2 copper layers, 0 parts

Commit message: LED done
Parts:
- added D1: LED_MINT, layout:LED_0603_Symbol_on_F.SilkS, F.Cu at (133.8, 90.0)
- added J1: Conn_01x02, Connector_Molex:Molex_KK-254_AE-6410-02A_1x02_P2.54mm_Vertical, F.Cu at (134.5, 96.0)
- added R1: 105, Resistor_SMD:R_0603_1608Metric_Pad0.98x0.95mm_HandSolder, F.Cu at (138.0, 90.0)
- added REF**: MountingHole_3.2mm_M3, MountingHole:MountingHole_3.2mm_M3, F.Cu at (135.0, 85.0)
- added REF**: MountingHole_3.2mm_M3, MountingHole:MountingHole_3.2mm_M3, F.Cu at (144.2, 97.2)
- added SW1: SW_Push, Button_Switch_SMD:SW_DIP_SPSTx01_Slide_6.7x4.1mm_W8.61mm_P2.54mm_LowProfile, F.Cu at (144.0, 87.0)
Routing:
- net Net-(R1-Pad1): track 0.00 -> 11.3 mm
- net Net-(D1-A): track 0.00 -> 2.49 mm
- net GND: track 0.00 -> 1.60 mm, vias 0 -> 1
- added copper zone on F.Cu, net +3V3
- added copper zone on B.Cu, net GND
Other:
- board outline added: 17 x 21 mm
