File: Hardware/Dev/Template_v0.0/LED/LED.kicad_sch (KiCad schematic)
At the start: 0 parts

Commit message: first commit
Parts:
- added D1: LED_MINT, layout:LED_0603_Symbol_on_F.SilkS, symbol device:LED
- added J1: Conn_01x02, Connector_Molex:Molex_KK-254_AE-6410-02A_1x02_P2.54mm_Vertical, symbol Connector_Generic:Conn_01x02
- added R1: 105, Resistor_SMD:R_0603_1608Metric_Pad0.98x0.95mm_HandSolder, symbol device:R_US
- added SW1: SW_Push, Button_Switch_SMD:SW_DIP_SPSTx01_Slide_6.7x4.1mm_W8.61mm_P2.54mm_LowProfile, symbol Switch:SW_Push
Connections:
- new net: R1.1, SW1.2
- new net: D1.2 (A), R1.2
- new net +3V3: J1.2 (Pin_2), SW1.1
- new net GND: D1.1 (K), J1.1 (Pin_1)
Other:
- title: Template -> LED Project

Commit message: LED done
Parts:
- J1: MPN (none) -> 022272021
- SW1: MPN (none) -> 1825910-6
Changed lines of the file:
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@@
       (effects (font (size 1.27 1.27)) hide)
     )
-    (property "Datasheet" "~" (at 72.39 69.85 0)
+    (property "Datasheet" "https://www.te.com/usa-en/product-1825910-6.datasheet.pdf" (at 72.39 69.85 0)
+      (effects (font (size 1.27 1.27)) hide)
+    )
+    (property "MPN" "1825910-6" (at 72.39 74.93 0)
       (effects (font (size 1.27 1.27)) hide)
     )
@@
       (effects (font (size 1.27 1.27)) hide)
     )
+    (property "MPN" "" (at 96.52 83.82 0)
+      (effects (font (size 1.27 1.27)) hide)
+    )
     (pin "1")
     (pin "2")
@@
       (effects (font (size 1.27 1.27)) hide)
     )
+    (property "MPN" "" (at 87.63 74.93 0)
+      (effects (font (size 1.27 1.27)) hide)
+    )
     (pin "1")
     (pin "2")
@@
       (effects (font (size 1.27 1.27)) hide)
     )
-    (property "Datasheet" "~" (at 49.53 86.36 0)
+    (property "Datasheet" "https://tools.molex.com/pdm_docs/sd/022272021_sd.pdf" (at 49.53 86.36 0)
       (effects (font (size 1.27 1.27)) hide)
     )
+    (property "MPN" "022272021" (at 49.53 86.36 0)
+      (effects (font (size 1.27 1.27)) hide)
+    )
