File: Hardware/horns/horns.kicad_sch (KiCad schematic)
At the start: 0 parts

Commit message: starting schematic
Parts:
- added J1: Conn_01x03, symbol Connector_Generic:Conn_01x03
- added J2, J3: Conn_01x02, symbol Connector_Generic:Conn_01x02
Other:
- title: Template -> Horns
Changed lines of the file:
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@@
-(kicad_sch (version 20211123) (generator eeschema)
+(kicad_sch (version 20230121) (generator eeschema)
   (paper "USLetter")
   (title_block
-    (title "Template")
+    (title "Horns")
     (date "2022-08-16")
     (rev "0.0")
     (company "Illini Solar Car")
-    (comment 1 "Designed By: Your Name")
+    (comment 1 "Designed By: Dylan M")
+  )
+  (symbol (lib_id "Connector_Generic:Conn_01x02") (at 81.28 91.44 0) (unit 1)
+    (in_bom yes) (on_board yes) (dnp no) (fields_autoplaced)
+    (property "Reference" "J3" (at 83.82 91.44 0)
+      (effects (font (size 1.27 1.27)) (justify left))
+    )
+    (property "Value" "Conn_01x02" (at 83.82 93.98 0)
+      (effects (font (size 1.27 1.27)) (justify left))
+    )
+    (property "Footprint" "" (at 81.28 91.44 0)
+      (effects (font (size 1.27 1.27)) hide)
+    )
+    (property "Datasheet" "~" (at 81.28 91.44 0)
+      (effects (font (size 1.27 1.27)) hide)
+    )
+    (pin "1")
+    (pin "2")
+    (instances
+      (project "horns"
+        (path "/1e1b062d-fad0-427c-a622-c5b8a80b5268"
+          (reference "J3") (unit 1)
+        )
+      )
+    )
+  )
+  (symbol (lib_id "Connector_Generic:Conn_01x03") (at 81.28 69.85 0) (unit 1)
+    (in_bom yes) (on_board yes) (dnp no) (fields_autoplaced)
+    (property "Reference" "J1" (at 83.82 68.58 0)
+      (effects (font (size 1.27 1.27)) (justify left))
+    )
+    (property "Value" "Conn_01x03" (at 83.82 71.12 0)
+      (effects (font (size 1.27 1.27)) (justify left))
+    )
+    (property "Footprint" "" (at 81.28 69.85 0)
+      (effects (font (size 1.27 1.27)) hide)
+    )
+    (property "Datasheet" "~" (at 81.28 69.85 0)
+      (effects (font (size 1.27 1.27)) hide)
+    )
+    (pin "1")
+    (pin "2")
+    (pin "3")
+    (instances
+      (project "horns"
+        (path "/1e1b062d-fad0-427c-a622-c5b8a80b5268"
+          (reference "J1") (unit 1)
+        )
+      )
+    )
+  )
+  (symbol (lib_id "Connector_Generic:Conn_01x02") (at 81.28 82.55 0) (unit 1)
+    (in_bom yes) (on_board yes) (dnp no) (fields_autoplaced)
+    (property "Reference" "J2" (at 83.82 82.55 0)
+      (effects (font (size 1.27 1.27)) (justify left))
+    )
+    (property "Value" "Conn_01x02" (at 83.82 85.09 0)
+      (effects (font (size 1.27 1.27)) (justify left))
+    )
+    (property "Footprint" "" (at 81.28 82.55 0)
+      (effects (font (size 1.27 1.27)) hide)
+    )
+    (property "Datasheet" "~" (at 81.28 82.55 0)
+      (effects (font (size 1.27 1.27)) hide)
+    )
+    (pin "1")
+    (pin "2")
+    (instances
+      (project "horns"
+        (path "/1e1b062d-fad0-427c-a622-c5b8a80b5268"
+          (reference "J2") (unit 1)
+        )
+      )
+    )
   )
   (sheet_instances
