File: Hardware/emreta2_Horn/emreta2_Horn.kicad_sch (KiCad schematic)
At the start: 0 parts

Commit message: Added features described in Horn spec file to schematic file
Parts:
- added C1, C2, C3, C4: 0.1uF, Capacitor_SMD:C_0603_1608Metric_Pad1.08x0.95mm_HandSolder, symbol device:C
- added C5, C6: 1uF, Capacitor_SMD:C_0603_1608Metric_Pad1.08x0.95mm_HandSolder, symbol device:C
- added C7, C8: 10uF, Capacitor_SMD:C_0603_1608Metric_Pad1.08x0.95mm_HandSolder, symbol device:C
- added C9: 100uF, Capacitor_THT:CP_Radial_D10.0mm_P5.00mm, symbol device:C_Polarized_US
- added D1: ES2DA-13-F, Diode_SMD:D_1206_3216Metric_Pad1.42x1.75mm_HandSolder, symbol pspice:DIODE
- added D2: LED, LED_SMD:LED_0603_1608Metric_Pad1.05x0.95mm_HandSolder, symbol device:LED
- added F1: 2A Fuse, Fuse:Fuse_1206_3216Metric_Pad1.42x1.75mm_HandSolder, symbol device:Fuse
- added J1: Conn_01x03, Connector_Molex:Molex_KK-254_AE-6410-03A_1x03_P2.54mm_Vertical, symbol Connector_Generic:Conn_01x03
- added J2, J3, J4: Conn_01x02, Connector_Molex:Molex_KK-254_AE-6410-02A_1x02_P2.54mm_Vertical, symbol Connector_Generic:Conn_01x02
- added Q2: IRFR010PBF, Package_DirectFET:DirectFET_MT, symbol device:Q_NMOS_GDS
- added R1, R2: 1K, Resistor_SMD:R_0603_1608Metric_Pad0.98x0.95mm_HandSolder, symbol device:R_US
Connections:
- new net: F1.1, Q2.2 (D)
- new net: J3.2 (Pin_2), J4.1 (Pin_1)
- new net: D2.1 (K), R2.2
- new net +24V: C2.2, C3.2, C4.2, C5.2, C6.2, C7.2, C8.2, C9.1, D1.2 (A), J1.2 (Pin_2), J3.1 (Pin_1)
- new net GND: C1.1, C2.1, C3.1, C4.1, C5.1, C6.1, C7.1, C8.1, C9.2, J1.1 (Pin_1), J1.3 (Pin_3), J2.1 (Pin_1), Q2.3 (S), R1.1, R2.1
- new net HORN_CONTROL: C1.2, D2.2 (A), J2.2 (Pin_2), Q2.1 (G), R1.2
- new net HORN_IN: D1.1 (K), F1.2, J4.2 (Pin_2)
