File: Hardware/emreta2_Horn/emreta2_Horn.kicad_pcb (KiCad board)
At the start: 2 copper layers, 0 parts

Commit message: Designed Layout, made changes to 'emreta2_Horn.md' in the test points section, added three test points that were not in the schematic.
Parts:
- added C1: 0.1uF, Capacitor_SMD:C_0603_1608Metric_Pad1.08x0.95mm_HandSolder, F.Cu at (68.0, 103.1)
- added C2: 0.1uF, Capacitor_SMD:C_0603_1608Metric_Pad1.08x0.95mm_HandSolder, F.Cu at (82.5, 92.0)
- added C3: 0.1uF, Capacitor_SMD:C_0603_1608Metric_Pad1.08x0.95mm_HandSolder, F.Cu at (82.5, 93.9)
- added C4: 0.1uF, Capacitor_SMD:C_0603_1608Metric_Pad1.08x0.95mm_HandSolder, F.Cu at (82.5, 95.9)
- added C5: 1uF, Capacitor_SMD:C_0603_1608Metric_Pad1.08x0.95mm_HandSolder, F.Cu at (82.5, 97.8)
- added C6: 1uF, Capacitor_SMD:C_0603_1608Metric_Pad1.08x0.95mm_HandSolder, F.Cu at (82.5, 99.7)
- added C7: 10uF, Capacitor_SMD:C_0603_1608Metric_Pad1.08x0.95mm_HandSolder, F.Cu at (62.8, 88.3)
- added C8: 10uF, Capacitor_SMD:C_0603_1608Metric_Pad1.08x0.95mm_HandSolder, F.Cu at (66.6, 88.3)
- added C9: 100uF, Capacitor_THT:CP_Radial_D10.0mm_P5.00mm, F.Cu at (67.8, 92.4)
- added D1: ES2DA-13-F, Diode_SMD:D_1206_3216Metric_Pad1.42x1.75mm_HandSolder, F.Cu at (78.2, 91.8)
- added D2: LED, LED_SMD:LED_0603_1608Metric_Pad1.05x0.95mm_HandSolder, F.Cu at (62.9, 103.1)
- added F1: 2A Fuse, Fuse:Fuse_1206_3216Metric_Pad1.42x1.75mm_HandSolder, F.Cu at (76.1, 98.6)
- added HORN_CONNECTION: TestPoint_Pad_1.0x1.0mm, TestPoint:TestPoint_Pad_1.0x1.0mm, F.Cu at (69.5, 86.6)
- added HORN_CONTROL: TestPoint_Pad_1.0x1.0mm, TestPoint:TestPoint_Pad_1.0x1.0mm, F.Cu at (78.3, 102.5)
- added HORN_IN: TestPoint_Pad_1.0x1.0mm, TestPoint:TestPoint_Pad_1.0x1.0mm, F.Cu at (78.0, 95.5)
- added J1: Conn_01x03, Connector_Molex:Molex_KK-254_AE-6410-03A_1x03_P2.54mm_Vertical, F.Cu at (58.5, 98.1)
- added J2: Conn_01x02, Connector_Molex:Molex_KK-254_AE-6410-02A_1x02_P2.54mm_Vertical, F.Cu at (58.5, 105.0)
- added J3: Conn_01x02, Connector_Molex:Molex_KK-254_AE-6410-02A_1x02_P2.54mm_Vertical, F.Cu at (73.0, 86.3)
- added J4: Conn_01x02, Connector_Molex:Molex_KK-254_AE-6410-02A_1x02_P2.54mm_Vertical, F.Cu at (79.7, 86.3)
- added Q1: IRFR010PBF, Package_DirectFET:DirectFET_MT, F.Cu at (73.2, 104.4)
- added R1: 1K, Resistor_SMD:R_0603_1608Metric_Pad0.98x0.95mm_HandSolder, F.Cu at (65.5, 103.1)
- added R2: 1K, Resistor_SMD:R_0603_1608Metric_Pad0.98x0.95mm_HandSolder, F.Cu at (64.8, 105.8)
- added REF**: MountingHole_3.2mm_M3, MountingHole:MountingHole_3.2mm_M3, F.Cu at (82.5, 104.8)
- added REF**: MountingHole_3.2mm_M3, MountingHole:MountingHole_3.2mm_M3, F.Cu at (57.1, 85.7)
Routing:
- net GND: track 0.00 -> 28.1 mm, vias 0 -> 4
- net /HORN_CONTROL: track 0.00 -> 26.3 mm
- net /HORN_IN: track 0.00 -> 17.8 mm
- net Net-(J3-Pin_2): track 0.00 -> 16.1 mm
- net Net-(Q2-D): track 0.00 -> 6.95 mm
- net Net-(D2-K): track 0.00 -> 2.71 mm
- added copper zone on F.Cu, net +24V
- added copper zone on B.Cu, net GND
Other:
- board outline added: 31.7 x 25.4 mm
