File: Hardware/proj_1_LED/proj_1_LED.kicad_pcb (KiCad board)
At the start: 2 copper layers, 0 parts

Commit message: Nearly finish LED project
Parts:
- added D1: LED_GREEN, layout:LED_0603_Symbol_on_F.SilkS, F.Cu at (44.5, 27.5)
- added J1: Conn_01x02, Connector_Molex:Molex_KK-254_AE-6410-02A_1x02_P2.54mm_Vertical, F.Cu at (43.2, 34.0)
- added R1: 105, Resistor_SMD:R_0201_0603Metric_Pad0.64x0.40mm_HandSolder, F.Cu at (37.6, 34.6)
- added REF**: MountingHole_3.2mm_M3, MountingHole:MountingHole_3.2mm_M3, F.Cu at (44.5, 44.5)
- added REF**: MountingHole_3.2mm_M3, MountingHole:MountingHole_3.2mm_M3, F.Cu at (37.5, 29.0)
- added SW1: SW_Push, Button_Switch_SMD:SW_DIP_SPSTx01_Slide_6.7x4.1mm_W8.61mm_P2.54mm_LowProfile, F.Cu at (37.5, 42.5)
Routing:
- net Net-(D1-A): track 0.00 -> 21.8 mm
- net Net-(R1-Pad2): track 0.00 -> 3.61 mm
- net GND: track 0.00 -> 1.54 mm, vias 0 -> 1
- added copper zone on F.Cu, net +3V3
- added copper zone on B.Cu, net GND
Other:
- board outline added: 15.5 x 26 mm
