File: Hardware/Dev/Template_v0.0/Template_v0.0.kicad_pcb (KiCad board)
At the start: 2 copper layers, 0 parts

Commit message: haha
Parts:
- added D1: LED_RED, layout:LED_0603_Symbol_on_F.SilkS, F.Cu at (114.8, 50.5)
- added J1: Conn_01x02, Connector_Molex:Molex_KK-254_AE-6410-02A_1x02_P2.54mm_Vertical, F.Cu at (115.2, 55.5)
- added R1: 105, Resistor_SMD:R_0603_1608Metric_Pad0.98x0.95mm_HandSolder, F.Cu at (119.9, 50.0)
- added REF**: MountingHole_3.2mm_M3, MountingHole:MountingHole_3.2mm_M3, F.Cu at (123.5, 55.5)
- added REF**: MountingHole_3.2mm_M3, MountingHole:MountingHole_3.2mm_M3, F.Cu at (117.0, 45.0)
- added SW1: SW_Push, Button_Switch_SMD:SW_DIP_SPSTx01_Slide_6.7x4.1mm_W8.61mm_P2.54mm_LowProfile, F.Cu at (124.5, 45.5)
Routing:
- net Net-(R1-Pad2): track 0.00 -> 10.9 mm
- net Net-(D1-A): track 0.00 -> 3.61 mm
- net GND: track 0.00 -> 1.25 mm, vias 0 -> 1
- added copper zone on F.Cu, net +3V3
- added copper zone on B.Cu, net GND
