File: Hardware/Dev/Template_v0.0/Template_v0.0.kicad_pcb (KiCad board)
At the start: 2 copper layers, 0 parts

Commit message: Firmware Projects1 & 2
Parts:
- added D1: LED_BLUE, layout:LED_0603_Symbol_on_F.SilkS, F.Cu at (113.7, 99.5)
- added J1: Conn_01x02, Connector_Molex:Molex_KK-254_AE-6410-02A_1x02_P2.54mm_Vertical, F.Cu at (118.0, 97.5)
- added R1: 1K, Resistor_SMD:R_0603_1608Metric_Pad0.98x0.95mm_HandSolder, F.Cu at (113.6, 95.0)
- added REF**: MountingHole_3.2mm_M3, MountingHole:MountingHole_3.2mm_M3, F.Cu at (121.5, 89.0)
- added REF**: MountingHole_3.2mm_M3, MountingHole:MountingHole_3.2mm_M3, F.Cu at (108.0, 97.0)
- added SW1: SW_Push, Button_Switch_SMD:SW_DIP_SPSTx01_Slide_6.7x4.1mm_W8.61mm_P2.54mm_LowProfile, F.Cu at (111.5, 89.0)
Routing:
- net Net-(R1-Pad1): track 0.00 -> 7.30 mm
- net Net-(D1-A): track 0.00 -> 4.50 mm
- net GND: track 0.00 -> 1.96 mm, vias 0 -> 1
- added copper zone on F.Cu, net +3V3
- added copper zone on B.Cu, net GND
Other:
- board outline added: 22.1 x 19.2 mm
