File: Hardware/Dev/Template_v0.0/Template_v0.0.kicad_pcb (KiCad board)
At the start: 2 copper layers, 0 parts

Commit message: moving hardware files to ./hardware
Parts:
- added D1: LED_RED, layout:LED_0603_Symbol_on_F.SilkS, F.Cu at (120.3, 70.1)
- added J1: Conn_01x02, Connector_Molex:Molex_KK-254_AE-6410-02A_1x02_P2.54mm_Vertical, F.Cu at (122.5, 76.5)
- added R1: 105, Resistor_SMD:R_0603_1608Metric_Pad0.98x0.95mm_HandSolder, F.Cu at (125.4, 69.8)
- added REF**: MountingHole_3.2mm_M3, MountingHole:MountingHole_3.2mm_M3, F.Cu at (132.0, 77.0)
- added REF**: MountingHole_3.2mm_M3, MountingHole:MountingHole_3.2mm_M3, F.Cu at (122.0, 63.0)
- added SW1: SW_Push, Button_Switch_SMD:SW_DIP_SPSTx01_Slide_6.7x4.1mm_W8.61mm_P2.54mm_LowProfile, F.Cu at (131.0, 65.0)
Routing:
- net Net-(R1-Pad1): track 0.00 -> 12.6 mm
- net Net-(D1-A): track 0.00 -> 3.51 mm
- net GND: track 0.00 -> 2.20 mm, vias 0 -> 1
- added copper zone on F.Cu, net +3V3
- added copper zone on B.Cu, net GND
Other:
- board outline added: 24.5 x 26 mm
