File: Hardware/Dev/Template_v0.0/Template_v0.0.kicad_sch (KiCad schematic)
At the start: 0 parts

Commit message: proj 1
Other:
- title: Template -> Proj 1
Changed lines of the file:
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@@
 	(paper "USLetter")
 	(title_block
-		(title "Template")
+		(title "Proj 1")
 		(date "2022-08-16")
 		(rev "0.0")
 		(company "Illini Solar Car")
-		(comment 1 "Designed By: Your Name")
+		(comment 1 "Designed By: Enrique Garcia - eg20")
 	)
 	(sheet_instances
