File: Hardware/Dev/Template_v0.0/Template_v0.0.kicad_sch (KiCad schematic)
At the start: 0 parts

Commit message: Merged changes from origin.
Parts:
- added D1: LED, symbol Device:LED
- added J1: Conn_01x02, symbol Connector_Generic:Conn_01x02
- added R1: R, symbol Device:R
- added SW1: SW_Push, symbol Switch:SW_Push
Connections:
- new net +3V3: J1.1 (Pin_1)
- new net GND: J1.2 (Pin_2)

Commit message: Finished LED Project
Parts:
- D1: footprint (none) -> layout:LED_0603_Symbol_on_F.SilkS
- J1: footprint (none) -> Connector_Molex:Molex_KK-254_AE-6410-02A_1x02_P2.54mm_Vertical; MPN (none) -> 022272021
- R1: value R -> 1k; footprint (none) -> Resistor_SMD:R_0603_1608Metric_Pad0.98x0.95mm_HandSolder
- SW1: footprint (none) -> Button_Switch_SMD:SW_DIP_SPSTx01_Slide_6.7x4.1mm_W8.61mm_P2.54mm_LowProfile; MPN (none) -> 1825910-6
Connections:
- net +3V3: now also R1.1
- net GND: now also SW1.1
- net at D1.1 (K): now also SW1.2
- net at D1.2 (A): now also R1.2
Other:
- title: Template -> LED Project
