File: Hardware/HornsBoard_v1.0/HornsBoard_v1.0.kicad_sch (KiCad schematic)
At the start: 0 parts

Commit message: calumnd2 horns board schematic progress (incomplete)
Parts:
- added C1, C2, C3, C4: .1u, Capacitor_SMD:C_0201_0603Metric_Pad0.64x0.40mm_HandSolder, symbol Device:C
- added C5, C6: 1u, Capacitor_SMD:C_0201_0603Metric_Pad0.64x0.40mm_HandSolder, symbol Device:C
- added C7, C8: 10u, Capacitor_SMD:C_0201_0603Metric_Pad0.64x0.40mm_HandSolder, symbol Device:C
- added C9: C_Polarized_Small_US, symbol device:C_Polarized_Small_US
- added D1: ES2DA-13-F, symbol device:D
- added F1: 2, symbol device:Fuse
- added J1: Conn_01x03, symbol Connector_Generic:Conn_01x03
- added J2, J3, J4: Conn_01x02, symbol Connector_Generic:Conn_01x02
- added Q1: IRFR010PBF, Package_TO_SOT_SMD:TO-252-2, symbol Transistor_FET:QM6006D
- added R1: 1K, Resistor_SMD:R_0603_1608Metric_Pad0.98x0.95mm_HandSolder, symbol device:R
Connections:
- new net: C1.2, Q1.1 (G)
- new net: F1.2, Q1.2 (D)
- new net: C1.1, R1.2
- new net: J3.1 (Pin_1), J4.2 (Pin_2)
- new net +24V: C2.1, C3.1, C4.1, C5.1, C6.1, C7.1, C8.1, C9.1, J1.2 (Pin_2), J4.1 (Pin_1)
- new net GND: C2.2, C3.2, C4.2, C5.2, C6.2, C7.2, C8.2, C9.2, D1.1 (K), J1.1 (Pin_1), J1.3 (Pin_3), J2.1 (Pin_1), Q1.3 (S)
- new net HORN_CTL: J2.2 (Pin_2), R1.1
- new net HORN_IN: D1.2 (A), F1.1, J3.2 (Pin_2)

Commit message: calumnd2 horns board layout
Parts:
- added TP1, TP2, TP3, TP4: TestPoint, TestPoint:TestPoint_Pad_D1.0mm, symbol Connector:TestPoint
- C1, C2, C3, C4: value .1u -> .1uF; footprint Capacitor_SMD:C_0201_0603Metric_Pad0.64x0.40mm_HandSolder -> Capacitor_SMD:C_0603_1608Metric_Pad1.08x0.95mm_HandSolder
- C5, C6: value 1u -> 1uF; footprint Capacitor_SMD:C_0201_0603Metric_Pad0.64x0.40mm_HandSolder -> Capacitor_SMD:C_0603_1608Metric_Pad1.08x0.95mm_HandSolder
- C7, C8: value 10u -> 10uF; footprint Capacitor_SMD:C_0201_0603Metric_Pad0.64x0.40mm_HandSolder -> Capacitor_SMD:C_0603_1608Metric_Pad1.08x0.95mm_HandSolder
- C9: footprint (none) -> Capacitor_SMD:CP_Elec_6.3x3
- CTL_1: renamed from J2; footprint (none) -> Connector_Molex:Molex_KK-254_AE-6410-02A_1x02_P2.54mm_Vertical
- D1: footprint (none) -> Diode_SMD:D_SMA-SMB_Universal_Handsoldering
- F1: value 2 -> 2A; footprint (none) -> Fuse:Fuse_0603_1608Metric_Pad1.05x0.95mm_HandSolder
- HORN_1: renamed from J3; footprint (none) -> Connector_Molex:Molex_KK-254_AE-6410-02A_1x02_P2.54mm_Vertical
- HORN_2: renamed from J4; footprint (none) -> Connector_Molex:Molex_KK-254_AE-6410-02A_1x02_P2.54mm_Vertical
- PWR_1: renamed from J1; footprint (none) -> Connector_Molex:Molex_KK-254_AE-6410-03A_1x03_P2.54mm_Vertical
Connections:
- net +24V: now also D1.1 (K), TP3.1
- net GND: now also TP4.1; no longer D1.1 (K)
- net HORN_CTL: now also TP1.1
- net HORN_IN: now also TP2.1
