File: Hardware/HornsBoard_v1.0/HornsBoard_v1.0.kicad_sch (KiCad schematic)
At the start: 20 parts, among them J1_HORN_IN1 Conn_01x03, J2_HORN_CTRL1 Conn_01x02, J3_HORN_OUT1 Conn_01x02, J4 Conn_01x02, Q1 Q_PMOS_DGS

Commit message: hardware challenge project push
Parts:
- removed C2: 0.1uF, symbol Device:C
- removed D1: MDB6S, Package_SO:TSSOP-4_4.4x5mm_P4mm, symbol Diode_Bridge:MDB6S
- removed Q1: Q_PMOS_DGS, symbol Device:Q_PMOS_DGS
- removed R2: 1k, symbol Device:R_US
- added D1: D_Schottky, Diode_SMD:Nexperia_CFP3_SOD-123W, symbol device:D_Schottky
- added Q1: Q_NMOS_DGS, Package_TO_SOT_SMD:TO-252-2, symbol device:Q_NMOS_DGS
- C1: footprint (none) -> Capacitor_SMD:C_0603_1608Metric_Pad1.08x0.95mm_HandSolder
- C2: renamed from C3; footprint (none) -> Capacitor_SMD:C_0603_1608Metric_Pad1.08x0.95mm_HandSolder
- C3: renamed from C4; footprint (none) -> Capacitor_SMD:C_0603_1608Metric_Pad1.08x0.95mm_HandSolder
- C4: renamed from C5; footprint (none) -> Capacitor_SMD:C_0603_1608Metric_Pad1.08x0.95mm_HandSolder
- C5: renamed from C6; footprint (none) -> Capacitor_SMD:C_0603_1608Metric_Pad1.08x0.95mm_HandSolder
- C6: renamed from C7; footprint (none) -> Capacitor_SMD:C_0603_1608Metric_Pad1.08x0.95mm_HandSolder
- C7: renamed from C8; footprint (none) -> Capacitor_SMD:C_0603_1608Metric_Pad1.08x0.95mm_HandSolder
- C8: renamed from C9; footprint (none) -> Capacitor_SMD:C_0603_1608Metric_Pad1.08x0.95mm_HandSolder
- C9: renamed from C10; footprint (none) -> Capacitor_SMD:C_0603_1608Metric_Pad1.08x0.95mm_HandSolder
- F1, F2: footprint (none) -> Fuse:Fuse_0603_1608Metric_Pad1.05x0.95mm_HandSolder
- J1: renamed from J1_HORN_IN1; footprint (none) -> Connector_Molex:Molex_KK-254_AE-6410-03A_1x03_P2.54mm_Vertical; MPN (none) -> 022272031; Notes (none) -> HORN_IN
- J2: renamed from J2_HORN_CTRL1; footprint (none) -> Connector_Molex:Molex_KK-254_AE-6410-02A_1x02_P2.54mm_Vertical; MPN (none) -> 022272021; Notes (none) -> HORN_CTL
- J3: renamed from J3_HORN_OUT1; footprint (none) -> Connector_Molex:Molex_KK-254_AE-6410-02A_1x02_P2.54mm_Vertical; MPN (none) -> 022272021; Notes (none) -> HORN_OUT
- J4: footprint (none) -> Connector_Molex:Molex_KK-254_AE-6410-02A_1x02_P2.54mm_Vertical; MPN (none) -> 022272021; Notes (none) -> HORN_OUT
- R1: footprint (none) -> Resistor_SMD:R_0603_1608Metric_Pad0.98x0.95mm_HandSolder
Connections:
- net +24V: now also C1.1, C3.1, C4.1, C5.1, C6.1, C7.1, C8.1, C9.1, D1.1 (K); no longer F2.2, J1.2 (Pin_2)
- net GND: now also C1.2, C2.2, C3.2, C4.2, C5.2, C6.2, C7.2, C8.2, C9.2, J1.3 (Pin_3), Q1.3 (S)
- net horn_ctrl: now reaches R1.1
- net horn_ctrl: now also C2.1, J2.2 (Pin_2); no longer C2.2
- net at F2.1: now also Q1.1 (D)
- net at F1.1: now also Q1.2 (G)
- net at J4.2 (Pin_2): now also F2.2
- new net: D1.2 (A), J1.2 (Pin_2)
Other:
- moved on the sheet: C2, F1, F2, J1, J2, J3, J4, R1
