File: Hardware/HornsBoard_v1.0/HornsBoard_v1.0.kicad_pcb (KiCad board)
At the start: 2 copper layers, 0 parts

Commit message: calumnd2 horns board layout
Parts:
- added C1: .1uF, Capacitor_SMD:C_0603_1608Metric_Pad1.08x0.95mm_HandSolder, F.Cu at (96.2, 35.2)
- added C2: .1uF, Capacitor_SMD:C_0603_1608Metric_Pad1.08x0.95mm_HandSolder, F.Cu at (108.9, 44.0)
- added C3: .1uF, Capacitor_SMD:C_0603_1608Metric_Pad1.08x0.95mm_HandSolder, F.Cu at (108.9, 42.2)
- added C4: .1uF, Capacitor_SMD:C_0603_1608Metric_Pad1.08x0.95mm_HandSolder, F.Cu at (108.9, 40.5)
- added C5: 1uF, Capacitor_SMD:C_0603_1608Metric_Pad1.08x0.95mm_HandSolder, F.Cu at (108.9, 38.8)
- added C6: 1uF, Capacitor_SMD:C_0603_1608Metric_Pad1.08x0.95mm_HandSolder, F.Cu at (108.9, 37.0)
- added C7: 10uF, Capacitor_SMD:C_0603_1608Metric_Pad1.08x0.95mm_HandSolder, F.Cu at (108.9, 35.2)
- added C8: 10uF, Capacitor_SMD:C_0603_1608Metric_Pad1.08x0.95mm_HandSolder, F.Cu at (108.9, 33.5)
- added C9: C_Polarized_Small_US, Capacitor_SMD:CP_Elec_6.3x3, F.Cu at (88.8, 35.5)
- added CTL_1: Conn_01x02, Connector_Molex:Molex_KK-254_AE-6410-02A_1x02_P2.54mm_Vertical, F.Cu at (99.8, 27.0)
- added D1: ES2DA-13-F, Diode_SMD:D_SMA-SMB_Universal_Handsoldering, F.Cu at (88.5, 43.5)
- added F1: 2A, Fuse:Fuse_0603_1608Metric_Pad1.05x0.95mm_HandSolder, F.Cu at (96.4, 43.5)
- added HORN_1: Conn_01x02, Connector_Molex:Molex_KK-254_AE-6410-02A_1x02_P2.54mm_Vertical, F.Cu at (92.6, 27.0)
- added HORN_2: Conn_01x02, Connector_Molex:Molex_KK-254_AE-6410-02A_1x02_P2.54mm_Vertical, F.Cu at (85.5, 27.0)
- added PWR_1: Conn_01x03, Connector_Molex:Molex_KK-254_AE-6410-03A_1x03_P2.54mm_Vertical, F.Cu at (78.0, 30.2)
- added Q1: IRFR010PBF, Package_TO_SOT_SMD:TO-252-2, F.Cu at (102.9, 38.9)
- added R1: 1K, Resistor_SMD:R_0603_1608Metric_Pad0.98x0.95mm_HandSolder, F.Cu at (96.2, 33.2)
- added REF**: MountingHole_3.2mm_M3, MountingHole:MountingHole_3.2mm_M3, F.Cu at (109.0, 26.5)
- added REF**: MountingHole_3.2mm_M3, MountingHole:MountingHole_3.2mm_M3, F.Cu at (78.0, 42.5)
- added TP1: TestPoint, TestPoint:TestPoint_Pad_D1.0mm, F.Cu at (105.5, 30.2)
- added TP2: TestPoint, TestPoint:TestPoint_Pad_D1.0mm, F.Cu at (97.1, 40.2)
- added TP3: TestPoint, TestPoint:TestPoint_Pad_D1.0mm, F.Cu at (77.2, 25.8)
- added TP4: TestPoint, TestPoint:TestPoint_Pad_D1.0mm, F.Cu at (80.5, 25.8)
Routing:
- net GND: track 0.00 -> 22.6 mm, vias 0 -> 3
- net /HORN_IN: track 0.00 -> 22.3 mm
- net /HORN_CTL: track 0.00 -> 12.9 mm
- net Net-(Q1-G): track 0.00 -> 8.88 mm
- net Net-(Q1-D): track 0.00 -> 6.65 mm
- net Net-(HORN_1-Pin_1): track 0.00 -> 4.57 mm
- net Net-(C1-Pad1): track 0.00 -> 2.07 mm
- added copper zone on F.Cu, net +24V
- added copper zone on B.Cu, net GND
Other:
- board outline added: 40 x 25 mm

Commit message: calumnd2 horns board gerbers & dfm
Parts:
- moved CTL_1 0.75 mm to (99.8, 27.8)
- moved HORN_1 0.75 mm to (92.6, 27.8)
- moved HORN_2 0.75 mm to (85.5, 27.8)
- moved Q1 0.60 mm to (102.9, 38.3)
- moved TP1 0.25 mm to (105.5, 30.5)
Routing:
- net /HORN_CTL: track 12.9 -> 12.0 mm
- net /HORN_IN: track 22.3 -> 21.5 mm
Changed lines of the file:
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@@
 		(allow_soldermask_bridges_in_footprints no)
 		(pcbplotparams
-			(layerselection 0x00010fc_ffffffff)
+			(layerselection 0x00010f0_ffffffff)
 			(plot_on_all_layers_selection 0x0000000_00000000)
 			(disableapertmacros no)
@@
 			(outputformat 1)
 			(mirror no)
-			(drillshape 1)
+			(drillshape 0)
 			(scaleselection 1)
-			(outputdirectory "")
+			(outputdirectory "gerbers/")
 		)
 	)
@@
 	(footprint "Package_TO_SOT_SMD:TO-252-2"
 		(layer "F.Cu")
-		(at 102.8875 38.925 -90)
+		(at 102.8875 38.3275 -90)
 		(descr "TO-252 / DPAK SMD package, http://www.infineon.com/cms/en/product/packages/PG-TO252/PG-TO252-3-1/")
 		(tags "DPAK TO-252 DPAK-3 TO-252-3 SOT-428")
@@
 	(footprint "Connector_Molex:Molex_KK-254_AE-6410-02A_1x02_P2.54mm_Vertical"
 		(layer "F.Cu")
-		(at 92.6 27.02)
+		(at 92.6 27.77)
 		(descr "Molex KK-254 Interconnect System, old/engineering part number: AE-6410-02A example for new part number: 22-27-2021, 2 Pins (http://www.molex.com/pdm_docs/sd/022272021_sd.pdf), generated with kicad-footprint-generator")
 		(tags "connector Molex KK-254 vertical")
@@
 		(tags "Diode Universal SMA (DO-214AC) SMB (DO-214AA) Handsoldering ")
 		(property "Reference" "D1"
-			(at -0.725 -3 0)
+			(at 0.0125 -3 0)
 			(layer "F.SilkS")
 			(effects
@@
 	(footprint "Connector_Molex:Molex_KK-254_AE-6410-02A_1x02_P2.54mm_Vertical"
 		(layer "F.Cu")
-		(at 85.5 27)
+		(at 85.5 27.75)
 		(descr "Molex KK-254 Interconnect System, old/engineering part number: AE-6410-02A example for new part number: 22-27-2021, 2 Pins (http://www.molex.com/pdm_docs/sd/022272021_sd.pdf), generated with kicad-footprint-generator")
 		(tags "connector Molex KK-254 vertical")
@@
 	(footprint "TestPoint:TestPoint_Pad_D1.0mm"
 		(layer "F.Cu")
-		(at 105.5 30.25 180)
+		(at 105.5 30.5 180)
 		(descr "SMD pad as test Point, diameter 1.0mm")
 		(tags "test point SMD pad")
@@
 		(tags "capacitor electrolytic")
 		(property "Reference" "C9"
-			(at 0 -4.35 0)
+			(at 0 -2.25 0)
 			(layer "F.SilkS")
 			(effects
@@
 	(footprint "Connector_Molex:Molex_KK-254_AE-6410-02A_1x02_P2.54mm_Vertical"
 		(layer "F.Cu")
-		(at 99.75 27)
+		(at 99.75 27.75)
 		(descr "Molex KK-254 Interconnect System, old/engineering part number: AE-6410-02A example for new part number: 22-27-2021, 2 Pins (http://www.molex.com/pdm_docs/sd/022272021_sd.pdf), generated with kicad-footprint-generator")
 		(tags "connector Molex KK-254 vertical")
@@
 	)
 	(segment
-		(start 98.15 36.15)
-		(end 97.25 35.25)
+		(start 97.415 35.5525)
+		(end 103.7425 35.5525)
 		(width 0.25)
 		(layer "F.Cu")
@@
 	)
 	(segment
-		(start 105.1675 34.725)
-		(end 103.7425 36.15)
+		(start 103.7425 35.5525)
+		(end 105.1675 34.1275)
 		(width 0.25)
 		(layer "F.Cu")
@@
 	)
 	(segment
-		(start 103.7425 36.15)
-		(end 98.15 36.15)
+		(start 97.1125 35.25)
+		(end 97.415 35.5525)
 		(width 0.25)
 		(layer "F.Cu")
@@
 	)
 	(segment
-		(start 100.6375 32.5)
-		(end 100.6375 34.695)
+		(start 100.6375 31.9025)
+		(end 100.6375 34.0975)
 		(width 0.25)
 		(layer "F.Cu")
@@
 	)
 	(via
-		(at 100.6375 32.5)
+		(at 100.6375 31.9025)
 		(size 0.8)
 		(drill 0.4)
@@
 	)
 	(segment
-		(start 95.14 27.02)
-		(end 96.25 28.13)
+		(start 95.14 27.77)
+		(end 96.25 28.88)
 		(width 0.25)
 		(layer "F.Cu")
@@
 	)
 	(segment
-		(start 96.25 28.13)
-		(end 96.25 39.3625)
+		(start 96.25 39.3625)
+		(end 96.25 28.88)
 		(width 0.25)
 		(layer "F.Cu")
@@
 	)
 	(segment
-		(start 97.2625 43.5)
-		(end 100.4125 43.5)
+		(start 102.8875 40.4275)
+		(end 99.815 43.5)
 		(width 0.25)
 		(layer "F.Cu")
@@
 	)
 	(segment
-		(start 100.4125 43.5)
-		(end 102.8875 41.025)
+		(start 99.815 43.5)
+		(end 97.2625 43.5)
 		(width 0.25)
 		(layer "F.Cu")
@@
 	)
 	(segment
-		(start 97.1625 32.1675)
-		(end 97.1625 33.25)
+		(start 97.1625 32.8775)
+		(end 102.29 27.75)
+		(width 0.25)
+		(layer "F.Cu")
+		(net 7)
+	)
+	(segment
+		(start 105.5 30.5)
+		(end 102.75 27.75)
 		(width 0.25)
 		(layer "F.Cu")
@@
 	)
 	(segment
-		(start 105.5 30.25)
-		(end 102.29 27.04)
+		(start 102.75 27.75)
+		(end 102.29 27.75)
 		(width 0.25)
 		(layer "F.Cu")
@@
 	)
 	(segment
-		(start 102.29 27)
-		(end 102.29 27.04)
+		(start 102.29 27.75)
+		(end 102.29 27.79)
 		(width 0.25)
 		(layer "F.Cu")
@@
 	)
 	(segment
-		(start 102.29 27.04)
-		(end 97.1625 32.1675)
+		(start 97.1625 33.25)
+		(end 97.1625 32.8775)
 		(width 0.25)
 		(layer "F.Cu")
@@
 	)
 	(segment
-		(start 92.58 27)
-		(end 92.6 27.02)
+		(start 92.58 27.75)
+		(end 92.6 27.77)
 		(width 0.25)
 		(layer "F.Cu")
@@
 	)
 	(segment
-		(start 88.04 27)
-		(end 92.58 27)
+		(start 88.04 27.75)
+		(end 92.58 27.75)
 		(width 0.25)
 		(layer "F.Cu")
