File: Hardware/HornsBoard_v1.0/HornsBoard_v1.0.kicad_pcb (KiCad board)
At the start: 2 copper layers, 0 parts

Commit message: hardware challenge project push
Parts:
- added C1: 100uF, Capacitor_SMD:C_0603_1608Metric_Pad1.08x0.95mm_HandSolder, F.Cu at (126.0, 85.0)
- added C2: 0.1uF, Capacitor_SMD:C_0603_1608Metric_Pad1.08x0.95mm_HandSolder, F.Cu at (134.1, 88.0)
- added C3: 0.1uF, Capacitor_SMD:C_0603_1608Metric_Pad1.08x0.95mm_HandSolder, F.Cu at (126.0, 88.0)
- added C4: 0.1uF, Capacitor_SMD:C_0603_1608Metric_Pad1.08x0.95mm_HandSolder, F.Cu at (126.0, 91.0)
- added C5: 0.1uF, Capacitor_SMD:C_0603_1608Metric_Pad1.08x0.95mm_HandSolder, F.Cu at (126.0, 94.0)
- added C6: 1uF, Capacitor_SMD:C_0603_1608Metric_Pad1.08x0.95mm_HandSolder, F.Cu at (130.0, 94.0)
- added C7: 1uF, Capacitor_SMD:C_0603_1608Metric_Pad1.08x0.95mm_HandSolder, F.Cu at (130.0, 91.0)
- added C8: 10uF, Capacitor_SMD:C_0603_1608Metric_Pad1.08x0.95mm_HandSolder, F.Cu at (130.0, 88.0)
- added C9: 10uF, Capacitor_SMD:C_0603_1608Metric_Pad1.08x0.95mm_HandSolder, F.Cu at (130.0, 85.0)
- added D1: D_Schottky, Diode_SMD:Nexperia_CFP3_SOD-123W, F.Cu at (134.5, 99.0)
- added F1: 2A, Fuse:Fuse_0603_1608Metric_Pad1.05x0.95mm_HandSolder, F.Cu at (134.0, 94.0)
- added F2: 2A, Fuse:Fuse_0603_1608Metric_Pad1.05x0.95mm_HandSolder, F.Cu at (134.0, 85.0)
- added J1: Conn_01x03, Connector_Molex:Molex_KK-254_AE-6410-03A_1x03_P2.54mm_Vertical, F.Cu at (140.6, 98.2)
- added J2: Conn_01x02, Connector_Molex:Molex_KK-254_AE-6410-02A_1x02_P2.54mm_Vertical, F.Cu at (138.7, 89.5)
- added J3: Conn_01x02, Connector_Molex:Molex_KK-254_AE-6410-02A_1x02_P2.54mm_Vertical, F.Cu at (142.5, 78.5)
- added J4: Conn_01x02, Connector_Molex:Molex_KK-254_AE-6410-02A_1x02_P2.54mm_Vertical, F.Cu at (133.8, 78.7)
- added Q1: Q_NMOS_DGS, Package_TO_SOT_SMD:TO-252-2, F.Cu at (150.2, 88.5)
- added R1: 1k, Resistor_SMD:R_0603_1608Metric_Pad0.98x0.95mm_HandSolder, F.Cu at (134.0, 91.0)
- added REF**: MountingHole_3.2mm_M3, MountingHole:MountingHole_3.2mm_M3, F.Cu at (153.0, 100.0)
- added REF**: MountingHole_3.2mm_M3, MountingHole:MountingHole_3.2mm_M3, F.Cu at (153.0, 77.0)
- added REF**: MountingHole_3.2mm_M3, MountingHole:MountingHole_3.2mm_M3, F.Cu at (127.0, 100.0)
- added REF**: MountingHole_3.2mm_M3, MountingHole:MountingHole_3.2mm_M3, F.Cu at (127.0, 77.0)
Routing:
- net GND: track 0.00 -> 31.3 mm, vias 0 -> 2
- net Net-(Q1-G): track 0.00 -> 22.0 mm
- net /horn_ctrl: track 0.00 -> 14.6 mm
- net Net-(D1-A): track 0.00 -> 14.4 mm
- net Net-(Q1-D): track 0.00 -> 11.6 mm
- net Net-(J4-Pin_2): track 0.00 -> 8.63 mm
- net Net-(F1-Pad2): track 0.00 -> 3.02 mm
- added copper zone on F.Cu, net +24V
- added copper zone on B.Cu, net GND
Other:
- board outline added: 34 x 31 mm
