File: Hardware/proj1/proj1.kicad_pcb (KiCad board)
At the start: 2 copper layers, 0 parts

Commit message: updated project1 done
Parts:
- added D1: LED_RED, layout:LED_0603_Symbol_on_F.SilkS, F.Cu at (116.0, 101.0)
- added J1: Conn_01x02, Connector_Molex:Molex_KK-254_AE-6410-02A_1x02_P2.54mm_Vertical, F.Cu at (116.7, 107.0)
- added R1: 105, Resistor_SMD:R_0603_1608Metric_Pad0.98x0.95mm_HandSolder, F.Cu at (121.1, 101.0)
- added REF**: MountingHole_3.2mm_M3, MountingHole:MountingHole_3.2mm_M3, F.Cu at (126.2, 107.6)
- added REF**: MountingHole_3.2mm_M3, MountingHole:MountingHole_3.2mm_M3, F.Cu at (117.9, 93.2)
- added SW1: SW_Push, Button_Switch_SMD:SW_DIP_SPSTx01_Slide_6.7x4.1mm_W8.61mm_P2.54mm_LowProfile, F.Cu at (126.5, 94.5)
Routing:
- net Net-(R1-Pad1): track 0.00 -> 14.7 mm
- net Net-(D1-A): track 0.00 -> 6.91 mm
- net GND: track 0.00 -> 2.07 mm, vias 0 -> 1
- added copper zone on F.Cu, net +3V3
- added copper zone on B.Cu, net GND
