File: Hardware/proj1/Template_v0.0.kicad_sch (KiCad schematic)
At the start: 0 parts

Commit message: finished the projects
Parts:
- added D1: LED_RED, symbol Device:LED
- added J1: Conn_01x02, symbol Connector_Generic:Conn_01x02
- added R1: 105, symbol device:R_US
- added SW1: SW_Push, symbol Switch:SW_Push
Connections:
- new net: D1.2 (A), R1.2
- new net: R1.1, SW1.2
- new net +3V3: J1.2 (Pin_2), SW1.1
- new net GND: D1.1 (K), J1.1 (Pin_1)
Other:
- title: Template -> LED Project
