File: Hardware/prog2/prog2.kicad_sch (KiCad schematic)
At the start: 0 parts

Commit message: added a few components
Parts:
- added C1: C, symbol Device:C
- added C2: C_Polarized, symbol device:C_Polarized
- added J1: Conn_01x03, symbol Connector_Generic:Conn_01x03
- added J2, J3, J4: Conn_01x02, symbol Connector_Generic:Conn_01x02
Other:
- title: Template -> Horns Board
