File: Hardware/Project 1/LED/Project 1.kicad_sch (KiCad schematic)
At the start: 4 parts, among them J1 Conn_01x02, SW1 SW_Push

Commit message: Firmware Projects1 & 2
Parts:
- removed R1: 1K, Resistor_SMD:R_0603_1608Metric_Pad0.98x0.95mm_HandSolder, symbol Device:R
- added R2: R, symbol Device:R
- D1: footprint layout:LED_0603_Symbol_on_F.SilkS -> (none); MPN 0603BBD0680S01 -> (none)
- J1: footprint Connector_Molex:Molex_KK-254_AE-6410-02A_1x02_P2.54mm_Vertical -> (none); MPN 022272021 -> (none)
- SW1: footprint Button_Switch_SMD:SW_DIP_SPSTx01_Slide_6.7x4.1mm_W8.61mm_P2.54mm_LowProfile -> (none); MPN 1825910-6 -> (none)
Connections:
- net +3V3: now also J1.1 (Pin_1); no longer J1.2 (Pin_2)
- net GND: now also J1.2 (Pin_2); no longer J1.1 (Pin_1)
- net at D1.2 (A): now also R2.2
- net at SW1.2: now also R2.1
