File: LED_Project/prog1.kicad_pcb (KiCad board)
At the start: 2 copper layers, 0 parts

Commit message: finished LED project
Parts:
- added D1: LED_RED, layout:LED_0603_Symbol_on_F.SilkS, F.Cu at (133.0, 87.0)
- added J1: Conn_01x02, Connector_Molex:Molex_KK-254_AE-6410-02A_1x02_P2.54mm_Vertical, F.Cu at (129.0, 85.0)
- added R2: 105, Resistor_SMD:R_0603_1608Metric_Pad0.98x0.95mm_HandSolder, F.Cu at (133.0, 83.0)
- added REF**: MountingHole_3.2mm_M3, MountingHole:MountingHole_3.2mm_M3, F.Cu at (138.0, 85.0)
- added REF**: MountingHole_3.2mm_M3, MountingHole:MountingHole_3.2mm_M3, F.Cu at (126.0, 77.5)
- added SW1: SW_Push, Button_Switch_SMD:SW_DIP_SPSTx01_Slide_6.7x4.1mm_W8.61mm_P2.54mm_LowProfile, F.Cu at (135.7, 77.5)
Routing:
- net Net-(R2-Pad1): track 0.00 -> 10.4 mm
- net +3V3: track 0.00 -> 9.54 mm
- net Net-(D1-A): track 0.00 -> 3.42 mm
- net GND: track 0.00 -> 1.08 mm, vias 0 -> 1
- added copper zone on F.Cu, net +3V3
- added copper zone on B.Cu, net GND
Other:
- board outline added: 20 x 16 mm
