File: Hardware/HornsBoard/HornsBoard.kicad_pcb (KiCad board)
At the start: 2 copper layers, 0 parts

Commit message: Finished Horns Board Project
Parts:
- added C1: .1 uF, Capacitor_SMD:CP_Elec_4x4.5, F.Cu at (151.9, 89.0)
- added C2: 1 uF, Capacitor_SMD:CP_Elec_4x4.5, F.Cu at (147.4, 101.8)
- added C3: .1 uF, Capacitor_SMD:CP_Elec_4x4.5, F.Cu at (147.4, 108.2)
- added C4: .1 uF, Capacitor_SMD:CP_Elec_4x4.5, F.Cu at (147.4, 115.2)
- added C5: 10 uF, Capacitor_SMD:CP_Elec_4x4.5, F.Cu at (139.2, 101.0)
- added C6: 1 uF, Capacitor_SMD:CP_Elec_4x4.5, F.Cu at (139.2, 109.0)
- added C7: .1 uF, Capacitor_SMD:CP_Elec_4x4.5, F.Cu at (131.7, 101.0)
- added C8: 10 uF, Capacitor_SMD:CP_Elec_4x4.5, F.Cu at (139.4, 94.5)
- added C9: 100 uF, Capacitor_SMD:CP_Elec_4x4.5, F.Cu at (147.4, 94.5)
- added D1: US2DA, Diode_SMD:D_SMA, F.Cu at (166.2, 119.2)
- added F1: 2A, Fuse:Fuse_0603_1608Metric, F.Cu at (165.0, 87.0)
- added J1: Conn_01x03, Connector_Molex:Molex_KK-396_A-41791-0003_1x03_P3.96mm_Vertical, F.Cu at (155.6, 109.8)
- added J2: Conn_01x02, Connector_Molex:Molex_KK-396_A-41791-0002_1x02_P3.96mm_Vertical, F.Cu at (137.5, 88.5)
- added J3: Conn_01x02, Connector_Molex:Molex_KK-396_A-41791-0002_1x02_P3.96mm_Vertical, F.Cu at (169.0, 109.2)
- added J4: Conn_01x02, Connector_Molex:Molex_KK-396_A-41791-0002_1x02_P3.96mm_Vertical, F.Cu at (168.2, 95.0)
- added Q1: BS108, Package_TO_SOT_THT:TO-92_Inline, F.Cu at (161.2, 86.5)
- added R1: 1 kOhm, Resistor_SMD:R_0201_0603Metric, F.Cu at (146.2, 81.5)
- added REF**: MountingHole_3.2mm_M3, MountingHole:MountingHole_3.2mm_M3, F.Cu at (139.5, 119.2)
- added REF**: MountingHole_3.2mm_M3, MountingHole:MountingHole_3.2mm_M3, F.Cu at (157.8, 96.5)
Routing:
- net GND: track 0.00 -> 61.6 mm, vias 0 -> 3
- net +24V: track 0.00 -> 26.1 mm
- net Net-(C6-Pad2): track 0.00 -> 26.1 mm
- net Net-(J3-Pin_1): track 0.00 -> 15.6 mm
- net Net-(Q1-G): track 0.00 -> 14.7 mm
- net /HornIn: track 0.00 -> 12.0 mm
- net Net-(C1-Pad1): track 0.00 -> 10.7 mm
- net /HornCtrl: track 0.00 -> 9.69 mm
- net Net-(C5-Pad2): track 0.00 -> 9.49 mm
- net Net-(J4-Pin_1): track 0.00 -> 9.04 mm
- net Net-(C8-Pad1): track 0.00 -> 8.93 mm
- net Net-(C2-Pad1): track 0.00 -> 8.74 mm
- net Net-(C3-Pad2): track 0.00 -> 8.49 mm
- net Net-(C5-Pad1): track 0.00 -> 8.09 mm
- net Net-(C2-Pad2): track 0.00 -> 7.99 mm
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- added copper zone on F.Cu, net +24V
- added copper zone on B.Cu, net GND
Other:
- board outline added: 49.8 x 45 mm
