File: Hardware/project2/project2_v0.0.kicad_pcb (KiCad board)
At the start: 2 copper layers, 0 parts

Commit message: finished layout and Instant DFM Report
Parts:
- added C1: 0.1uF, Capacitor_SMD:C_0603_1608Metric, F.Cu at (140.0, 101.0)
- added C2: 0.1uF, Capacitor_SMD:C_0603_1608Metric, F.Cu at (122.0, 101.0)
- added C3: 0.1uF, Capacitor_SMD:C_0603_1608Metric, F.Cu at (122.0, 104.0)
- added C4: 0.1uF, Capacitor_SMD:C_0603_1608Metric, F.Cu at (122.0, 107.0)
- added C5: 1uF, Capacitor_SMD:C_0603_1608Metric, F.Cu at (122.0, 111.0)
- added C6: 1uF, Capacitor_SMD:C_0603_1608Metric, F.Cu at (122.0, 114.0)
- added C7: 10uF, Capacitor_SMD:C_1206_3216Metric, F.Cu at (151.0, 97.0)
- added C8: 10uF, Capacitor_SMD:C_1206_3216Metric, F.Cu at (151.0, 100.0)
- added C9: 100uF, Capacitor_THT:C_Radial_D10.0mm_H20.0mm_P5.00mm, F.Cu at (143.5, 106.0)
- added D1: DIODE, Diode_SMD:D_SMA, F.Cu at (151.0, 92.0)
- added F1: 2A, Fuse:Fuse_0402_1005Metric, F.Cu at (137.6, 115.0)
- added J1: Conn_01x02, Connector_Molex:Molex_KK-254_AE-6410-02A_1x02_P2.54mm_Vertical, F.Cu at (128.5, 94.0)
- added J3: Conn_01x02, Connector_Molex:Molex_KK-254_AE-6410-02A_1x02_P2.54mm_Vertical, F.Cu at (135.5, 94.0)
- added J5: Conn_01x03, Connector_Molex:Molex_KK-396_5273-03A_1x03_P3.96mm_Vertical, F.Cu at (127.1, 107.0)
- added J6: Conn_01x02, Connector_Molex:Molex_KK-254_AE-6410-02A_1x02_P2.54mm_Vertical, F.Cu at (142.5, 94.0)
- added Q2: IRF7343PBF, Package_SO:SOIC-8_3.9x4.9mm_P1.27mm, F.Cu at (145.0, 115.0)
- added R1: 1k, Resistor_SMD:R_0603_1608Metric_Pad0.98x0.95mm_HandSolder, F.Cu at (139.3, 111.0)
- added REF**: MountingHole_2.1mm, MountingHole:MountingHole_2.1mm, F.Cu at (123.0, 91.0)
- added REF**: MountingHole_2.1mm, MountingHole:MountingHole_2.1mm, F.Cu at (152.0, 115.0)
Routing:
- net GND: track 0.00 -> 51.2 mm
- net /HORN_CTL: track 0.00 -> 24.0 mm
- net Net-(Q2A-G): track 0.00 -> 15.2 mm
- net +24V: track 0.00 -> 13.0 mm
- net Net-(F1-Pad2): track 0.00 -> 10.9 mm
- net Net-(J3-Pin_2): track 0.00 -> 8.18 mm
- net /HORN_IN: track 0.00 -> 7.37 mm
- added copper zone on F.Cu, net +24V
- added copper zone on B.Cu, net GND
Other:
- board outline added: 37 x 32 mm
