File: Hardware/LED_Project/LEDProject_v1.0.kicad_pcb (KiCad board)
At the start: 2 copper layers, 22 x 21 mm, 6 parts, among them J1 Conn_01x02, SW1 SW_Push

Commit message: Fixed LED ground connection & started second Firmware project
Routing:
- net GND: track 9.26 -> 0.00 mm
Changed lines of the file:
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@@
 		(net 1)
-	)
-	(segment
-		(start 117 109)
-		(end 118 109)
-		(width 0.25)
-		(layer "F.Cu")
-		(net 2)
-	)
-	(segment
-		(start 115.901573 107.901573)
-		(end 117 109)
-		(width 0.25)
-		(layer "F.Cu")
-		(net 2)
-	)
-	(segment
-		(start 119 110)
-		(end 120 109)
-		(width 0.25)
-		(layer "F.Cu")
-		(net 2)
-	)
-	(segment
-		(start 115.901573 105.52)
-		(end 115.901573 107.901573)
-		(width 0.25)
-		(layer "F.Cu")
-		(net 2)
-	)
-	(segment
-		(start 120 109)
-		(end 121.5 109)
-		(width 0.25)
-		(layer "F.Cu")
-		(net 2)
-	)
-	(segment
-		(start 118 109)
-		(end 119 110)
-		(width 0.25)
-		(layer "F.Cu")
-		(net 2)
 	)
 	(via

Commit message: LED ground connection tweak
Routing:
- net GND: track 0.00 -> 2.91 mm
Changed lines of the file:
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@@
 		(net 1)
+	)
+	(segment
+		(start 119 110)
+		(end 120 109)
+		(width 0.25)
+		(layer "F.Cu")
+		(net 2)
+	)
+	(segment
+		(start 120 109)
+		(end 121.5 109)
+		(width 0.25)
+		(layer "F.Cu")
+		(net 2)
 	)
 	(via
