File: Hardware/Libraries/Project_1/Project_1.kicad_pcb (KiCad board)
At the start: 2 copper layers, 6 parts, among them J1 Conn_01x02, SW1 SW_Push

Commit message: Project 1 Hardware I couldn't figure out why filled zone is not connected.
Routing:
- added copper zone on F.Cu, net +3V3
- added copper zone on B.Cu, net GND
Other:
- board outline added: 22 x 18.5 mm
Changed lines of the file:
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@@
 		(tags "SMD DIP Switch SPST Slide 8.61mm 338mil SMD LowProfile")
 		(property "Reference" "SW1"
-			(at 0.195 3.5 360)
+			(at 0.195 3.5 0)
 			(layer "F.SilkS")
 			(effects
@@
 		)
 		(property "Value" "SW_Push"
-			(at 0.195 -3.5 360)
+			(at 0.195 -3.5 0)
 			(layer "F.Fab")
 			(effects
@@
 		)
 		(property "Footprint" "Button_Switch_SMD:SW_DIP_SPSTx01_Slide_6.7x4.1mm_W8.61mm_P2.54mm_LowProfile"
-			(at 0 0 360)
+			(at 0 0 0)
 			(layer "F.Fab")
 			(hide yes)
@@
 		)
 		(property "Datasheet" "https://www.te.com/usa-en/product-1825910-6.datasheet.pdf"
-			(at 0 0 360)
+			(at 0 0 0)
 			(layer "F.Fab")
 			(hide yes)
@@
 		)
 		(property "Description" "Push button switch, generic, two pins"
-			(at 0 0 360)
+			(at 0 0 0)
 			(layer "F.Fab")
 			(hide yes)
@@
 		)
 		(fp_text user "on"
-			(at 0.4275 -1.3425 360)
+			(at 0.4275 -1.3425 0)
 			(layer "F.Fab")
 			(effects
@@
 		(tags "LED led 0603 SMD smd SMT smt smdled SMDLED smtled SMTLED")
 		(property "Reference" "D1"
-			(at 0 -1.25 360)
+			(at 0 -1.25 0)
 			(layer "F.SilkS")
 			(effects
@@
 		)
 		(property "Value" "LED_RED"
-			(at 0 1.35 360)
+			(at 0 1.35 0)
 			(layer "F.Fab")
 			(effects
@@
 		)
 		(property "Footprint" "layout:LED_0603_Symbol_on_F.SilkS"
-			(at 0 0 360)
+			(at 0 0 0)
 			(layer "F.Fab")
 			(hide yes)
@@
 		)
 		(property "Datasheet" ""
-			(at 0 0 360)
+			(at 0 0 0)
 			(layer "F.Fab")
 			(hide yes)
@@
 		)
 		(property "Description" "Light emitting diode"
-			(at 0 0 360)
+			(at 0 0 0)
 			(layer "F.Fab")
 			(hide yes)
@@
 		)
 	)
-	(gr_line
-		(start 133 72.5)
-		(end 133 86.5)
+	(gr_rect
+		(start 110.5 70.5)
+		(end 132.5 89)
 		(stroke
-			(width 0.15)
+			(width 0.2)
 			(type default)
 		)
-		(layer "F.Adhes")
-	)
-	(gr_line
-		(start 130.5 89)
-		(end 112.5 89)
-		(stroke
-			(width 0.15)
-			(type default)
-		)
-		(layer "F.Adhes")
-	)
-	(gr_arc
-		(start 112.5 89)
-		(mid 110.732233 88.267767)
-		(end 110 86.5)
-		(stroke
-			(width 0.15)
-			(type default)
-		)
-		(layer "F.Adhes")
-	)
-	(gr_line
-		(start 110 86.5)
-		(end 110 72.5)
-		(stroke
-			(width 0.15)
-			(type default)
-		)
-		(layer "F.Adhes")
-	)
-	(gr_arc
-		(start 110 72.5)
-		(mid 110.732233 70.732233)
-		(end 112.5 70)
-		(stroke
-			(width 0.15)
-			(type default)
-		)
-		(layer "F.Adhes")
-	)
-	(gr_arc
-		(start 130.5 70)
-		(mid 132.267767 70.732233)
-		(end 133 72.5)
-		(stroke
-			(width 0.15)
-			(type default)
-		)
-		(layer "F.Adhes")
-	)
-	(gr_arc
-		(start 133 86.5)
-		(mid 132.267767 88.267767)
-		(end 130.5 89)
-		(stroke
-			(width 0.15)
-			(type default)
-		)
-		(layer "F.Adhes")
-	)
-	(gr_line
-		(start 112.5 70)
-		(end 130.5 70)
-		(stroke
-			(width 0.15)
-			(type default)
-		)
-		(layer "F.Adhes")
+		(fill none)
+		(layer "Edge.Cuts")
 	)
 	(dimension
 		(type aligned)
-		(layer "B.Cu")
+		(layer "User.1")
 		(pts
-			(xy 110 70) (xy 110 89)
-		)
-		(height 9)
-		(gr_text "19.0000 mm"
-			(at 99.2 79.5 90)
-			(layer "B.Cu")
+			(xy 128.5 85) (xy 128.5 75.5)
+		)
+		(height 10)
+		(gr_text "9.5000 mm"
+			(at 136.7 80.25 90)
+			(layer "User.1")
 			(effects
 				(font
@@
 	(dimension
 		(type aligned)
-		(layer "B.Cu")
+		(layer "User.1")
 		(pts
-			(xy 110 89) (xy 133 89)
-		)
-		(height 9)
-		(gr_text "23.0000 mm"
-			(at 121.5 96.2 0)
-			(layer "B.Cu")
+			(xy 114.5 75.5) (xy 129 75.5)
+		)
+		(height -12)
+		(gr_text "14.5000 mm"
+			(at 121.75 61.7 0)
+			(layer "User.1")
 			(effects
 				(font
@@
 	(dimension
 		(type aligned)
-		(layer "Cmts.User")
+		(layer "User.1")
 		(pts
-			(xy 128.5 85) (xy 128.5 75.5)
-		)
-		(height 10)
-		(gr_text "9.5000 mm"
-			(at 136.7 80.25 90)
-			(layer "Cmts.User")
+			(xy 110 70) (xy 110 89)
+		)
+		(height 9)
+		(gr_text "19.0000 mm"
+			(at 99.2 79.5 90)
+			(layer "User.1")
 			(effects
 				(font
@@
 	(dimension
 		(type aligned)
-		(layer "Cmts.User")
+		(layer "User.1")
 		(pts
-			(xy 114.5 75.5) (xy 129 75.5)
-		)
-		(height -12)
-		(gr_text "14.5000 mm"
-			(at 121.75 61.7 0)
-			(layer "Cmts.User")
+			(xy 110 89) (xy 133 89)
+		)
+		(height 9)
+		(gr_text "23.0000 mm"
+			(at 121.5 96.2 0)
+			(layer "User.1")
 			(effects
 				(font
@@
 	)
 	(zone
-		(net 0)
-		(net_name "")
+		(net 3)
+		(net_name "+3V3")
 		(layer "F.Cu")
 		(hatch edge 0.5)
+		(priority 1)
 		(connect_pads
 			(clearance 0)
@@
 		(min_thickness 0.25)
 		(filled_areas_thickness no)
-		(keepout
-			(tracks allowed)
-			(vias allowed)
-			(pads not_allowed)
-			(copperpour allowed)
-			(footprints allowed)
-		)
 		(fill
 			(thermal_gap 0.5)
@@
 		(polygon
 			(pts
-				(xy 133 70) (xy 110 70) (xy 110 89) (xy 133 89)
+				(xy 110 70) (xy 133 70) (xy 133 89.5) (xy 110 89.5)
 			)
 		)
 	)
 	(zone
-		(net 0)
-		(net_name "")
+		(net 1)
+		(net_name "GND")
 		(layer "B.Cu")
 		(hatch edge 0.5)
@@
 		(min_thickness 0.25)
 		(filled_areas_thickness no)
-		(keepout
-			(tracks allowed)
-			(vias allowed)
-			(pads not_allowed)
-			(copperpour allowed)
-			(footprints allowed)
-		)
 		(fill
 			(thermal_gap 0.5)
@@
 		(polygon
 			(pts
-				(xy 110 70) (xy 133 70) (xy 133 89) (xy 110 89)
-			)
-		)
+				(xy 110 70) (xy 133 70) (xy 133 89.5) (xy 110 89.5)
+			)
+		)
